Commit message: minor fix

File: vault_description/urdf/box/box.urdf.xacro (robot description, xacro)
@@ -29,5 +29,5 @@
         </gazebo>
         <joint name="vault_box_joint" type="fixed">
-            <origin rpy="0 0 0" xyz="0 0 0"/>
+            <origin rpy="0 0 1.57" xyz="0 0 0"/>
             <parent link="${parent}" />
             <child link="vault_box_link" />
