Commit message: d435i + t265

File: vault_description/urdf/box/realsense_mount.urdf.xacro (robot description, xacro)
@@ -29,5 +29,5 @@
         </gazebo>
         <joint name="vault_realsense_mount_joint" type="fixed">
-            <origin rpy="0 0 0" xyz="0 -0.072 -0.0075"/>
+            <origin rpy="0 0 0" xyz="0 -0.075 -0.0225"/>
             <parent link="${parent}" />
             <child link="vault_realsense_mount_link" />

File: vault_description/urdf/sensors/gps/gps.urdf.xacro (robot description, xacro)
@@ -1,13 +1,13 @@
 <?xml version="1.0"?>
 <robot name="sensor_gps" xmlns:xacro="http://www.ros.org/wiki/xacro">
-  <xacro:macro name="sensor_gps" params="name parent *origin">
+  <xacro:macro name="sensor_gps" params="name namespace parent *origin">
     <!-- antenna -->
-    <joint name="${name}_antenna_joint" type="fixed">
+    <joint name="${namespace}_${name}_antenna_joint" type="fixed">
         <axis xyz="1 0 0"/>
         <xacro:insert_block name="origin"/>
         <parent link="${parent}"/>
-        <child link="${name}_antenna_link"/>
+        <child link="${namespace}_${name}_antenna_link"/>
     </joint>
-    <link name="${name}_antenna_link">
+    <link name="${namespace}_${name}_antenna_link">
       <inertial>
         <mass value="0.001"/>
@@ -29,9 +29,9 @@
       </collision>
     </link>
-    <gazebo reference="${name}_antenna_link">
+    <gazebo reference="${namespace}_${name}_antenna_link">
       <material>Gazebo/Grey</material>
     </gazebo>
     <!-- plugin -->
-    <gazebo reference="${name}_antenna_link">
+    <gazebo reference="${namespace}_${name}_antenna_link">
         <sensor name="gps_sensor" type="gps">
             <always_on>true</always_on>
@@ -39,7 +39,8 @@
             <plugin name="gps_controller" filename="libgazebo_ros_gps_sensor.so">
                 <ros>
+                    <namespace>${namespace}</namespace>
                     <remapping>gps_controller/out:=fix</remapping>
                 </ros>
-                <frame_name>${name}_antenna_link</frame_name>
+                <frame_name>${namespace}_${name}_antenna_link</frame_name>
             </plugin>
         </sensor>

File: vault_description/urdf/sensors/gps/gps_board.urdf.xacro (robot description, xacro)
@@ -1,13 +1,13 @@
 <?xml version="1.0"?>
 <robot name="gps_board" xmlns:xacro="http://www.ros.org/wiki/xacro">
-  <xacro:macro name="gps_board" params="name parent *origin">
+  <xacro:macro name="gps_board" params="name namespace parent *origin">
     <!-- board -->
-    <joint name="${name}_joint" type="fixed">
+    <joint name="${namespace}_${name}_joint" type="fixed">
         <axis xyz="1 0 0"/>
         <xacro:insert_block name="origin"/>
         <parent link="${parent}"/>
-        <child link="${name}_board_link"/>
+        <child link="${namespace}_${name}_board_link"/>
     </joint>
-    <link name="${name}_board_link">
+    <link name="${namespace}_${name}_board_link">
       <inertial>
         <mass value="0.001"/>
@@ -29,5 +29,5 @@
       </collision>
     </link>
-    <gazebo reference="${name}_board_link">
+    <gazebo reference="${namespace}_${name}_board_link">
       <material>Gazebo/Grey</material>
     </gazebo>

File: vault_description/urdf/sensors/hokuyo/hokuyo.urdf.xacro (robot description, xacro)
@@ -1,11 +1,11 @@
 <?xml version="1.0"?>
 <robot name="sensor_hokuyo" xmlns:xacro="http://www.ros.org/wiki/xacro">
-  <xacro:macro name="sensor_hokuyo" params="prefix parent *origin min_angle:=-1.57079637051 max_angle:=1.57079637051">
-    <joint name="${name}_base_joint" type="fixed">
+  <xacro:macro name="sensor_hokuyo" params="name namespace parent *origin min_angle:=-1.57079637051 max_angle:=1.57079637051">
+    <joint name="${namespace}_${name}_base_joint" type="fixed">
       <xacro:insert_block name="origin" />
       <parent link="${parent}"/>
-      <child link="${name}_base_link"/>
+      <child link="${namespace}_${name}_base_link"/>
     </joint>
-    <link name="${name}_base_link">
+    <link name="${namespace}_${name}_base_link">
       <collision>
         <origin xyz="0 0 -0.05" rpy="0 0 0"/>
@@ -26,15 +26,15 @@
       </inertial>
     </link>
-    <gazebo reference="${name}_base_link">
+    <gazebo reference="${namespace}_${name}_base_link">
         <material>Gazebo/DarkGrey</material>
     </gazebo>
-    <link name="${name}_link">
+    <link name="${namespace}_${name}_link">
     </link>
-    <joint name="${name}_joint" type="fixed">
-      <parent link="${name}_base_link"/>
-      <child link="${name}_link"/>
+    <joint name="${namespace}_${name}_joint" type="fixed">
+      <parent link="${namespace}_${name}_base_link"/>
+      <child link="${namespace}_${name}_link"/>
       <origin xyz="0.00 0 0.0" rpy="0 0 0"/>
     </joint>
-    <gazebo reference="${name}_link">
+    <gazebo reference="${namespace}_${name}_link">
             <sensor type="gpu_ray" name="hokuyo_sensor">
                 <pose>0 0 0 0 0 0</pose>
@@ -61,10 +61,11 @@
                     </noise>
                 </ray>
-                <plugin name="${name}_controller" filename="libgazebo_ros_ray_sensor.so">
+                <plugin name="${namespace}_${name}_controller" filename="libgazebo_ros_ray_sensor.so">
                   <ros>
+                    <namespace>${namespace}</namespace>
                     <remapping>~/out:=scan</remapping>
                   </ros>
                   <output_type>sensor_msgs/LaserScan</output_type>
-                  <frame_name>${name}_link</frame_name>
+                  <frame_name>${namespace}_${name}_link</frame_name>
                 </plugin>
             </sensor>

File: vault_description/urdf/sensors/imu/imu.urdf.xacro (robot description, xacro)
@@ -1,12 +1,12 @@
 <?xml version="1.0"?>
 <robot name="sensor_imu" xmlns:xacro="http://www.ros.org/wiki/xacro">
-  <xacro:macro name="sensor_imu" params="name parent *origin">
-    <joint name="${name}_joint" type="fixed">
+  <xacro:macro name="sensor_imu" params="name namespace parent *origin">
+    <joint name="${namespace}_${name}_joint" type="fixed">
         <axis xyz="1 0 0"/>
         <xacro:insert_block name="origin"/>
         <parent link="${parent}"/>
-        <child link="${name}_link"/>
+        <child link="${namespace}_${name}_link"/>
     </joint>
-    <link name="${name}_link">
+    <link name="${namespace}_${name}_link">
       <inertial>
         <mass value="0.001"/>
@@ -28,15 +28,16 @@
       </collision>
     </link>
-    <gazebo reference="${name}_link">
+    <gazebo reference="${namespace}_${name}_link">
         <material>Gazebo/Turquoise</material>
     </gazebo>
-    <gazebo reference="${name}_link">
+    <gazebo reference="${namespace}_${name}_link">
       <sensor name="imu_sensor" type="imu">
         <plugin filename="libgazebo_ros_imu_sensor.so" name="imu_controller">
           <ros>
+            <namespace>${namespace}</namespace>
             <remapping>~/out:=imu</remapping>
           </ros>
           <initial_orientation_as_reference>false</initial_orientation_as_reference>
-          <frame_name>${name}_link</frame_name>
+          <frame_name>${namespace}_${name}_link</frame_name>
         </plugin>
         <always_on>true</always_on>

File: vault_description/urdf/sensors/realsense/d435.urdf.xacro (robot description, xacro)
@@ -7,7 +7,6 @@
 -->
 <robot name="sensor_d435" xmlns:xacro="http://ros.org/wiki/xacro">
-  <xacro:macro name="sensor_d435" params="parent *origin name:=camera use_nominal_extrinsics:=false add_plug:=false use_mesh:=true">
+  <xacro:macro name="sensor_d435" params="parent *origin name:=d435 namespace:=vault use_nominal_extrinsics:=true add_plug:=false use_mesh:=true">
     <!-- Includes -->
-    <xacro:include filename="$(find vault_description)/urdf/sensors/realsense/materials.urdf.xacro" />
     <xacro:include filename="$(find vault_description)/urdf/sensors/realsense/usb_plug.urdf.xacro" />
     <xacro:property name="M_PI" value="3.1415926535897931" />
@@ -36,16 +35,16 @@
     <xacro:property name="d435_cam_depth_pz" value="${d435_cam_height/2}"/>
     <!-- camera body, with origin at bottom screw mount -->
-    <joint name="${name}_joint" type="fixed">
+    <joint name="${namespace}_${name}_joint" type="fixed">
       <xacro:insert_block name="origin" />
       <parent link="${parent}"/>
-      <child link="${name}_bottom_screw_frame" />
+      <child link="${namespace}_${name}_bottom_screw_frame" />
     </joint>
-    <link name="${name}_bottom_screw_frame"/>
-    <joint name="${name}_link_joint" type="fixed">
+    <link name="${namespace}_${name}_bottom_screw_frame"/>
+    <joint name="${namespace}_${name}_link_joint" type="fixed">
       <origin xyz="${d435_mesh_x_offset} ${d435_cam_depth_py} ${d435_cam_depth_pz}" rpy="0 0 0"/>
-      <parent link="${name}_bottom_screw_frame"/>
-      <child link="${name}_link" />
+      <parent link="${namespace}_${name}_bottom_screw_frame"/>
+      <child link="${namespace}_${name}_link" />
     </joint>
-    <link name="${name}_link">
+    <link name="${namespace}_${name}_link">
       <visual>
         <xacro:if value="${use_mesh}">
@@ -77,5 +76,5 @@
       </inertial>
     </link>
-    <gazebo reference="${name}_link">
+    <gazebo reference="${namespace}_${name}_link">
       <material>Gazebo/Silver</material>
     </gazebo>
@@ -83,68 +82,68 @@
     <xacro:if value="${use_nominal_extrinsics}">
       <!-- camera depth joints and links -->
-      <joint name="${name}_depth_joint" type="fixed">
+      <joint name="${namespace}_${name}_depth_joint" type="fixed">
         <origin xyz="0 0 0" rpy="0 0 0"/>
-        <parent link="${name}_link"/>
-        <child link="${name}_depth_frame" />
+        <parent link="${namespace}_${name}_link"/>
+        <child link="${namespace}_${name}_depth_frame" />
       </joint>
-      <link name="${name}_depth_frame"/>
-      <joint name="${name}_depth_optical_joint" type="fixed">
+      <link name="${namespace}_${name}_depth_frame"/>
+      <joint name="${namespace}_${name}_depth_optical_joint" type="fixed">
         <origin xyz="0 0 0" rpy="${-M_PI/2} 0 ${-M_PI/2}" />
-        <parent link="${name}_depth_frame" />
-        <child link="${name}_depth_optical_frame" />
+        <parent link="${namespace}_${name}_depth_frame" />
+        <child link="${namespace}_${name}_depth_optical_frame" />
       </joint>
-      <link name="${name}_depth_optical_frame"/>
+      <link name="${namespace}_${name}_depth_optical_frame"/>
       <!-- camera left IR joints and links -->
-      <joint name="${name}_infra1_joint" type="fixed">
+      <joint name="${namespace}_${name}_infra1_joint" type="fixed">
         <origin xyz="0 ${d435_cam_depth_to_infra1_offset} 0" rpy="0 0 0" />
-        <parent link="${name}_link" />
-        <child link="${name}_infra1_frame" />
+        <parent link="${namespace}_${name}_link" />
+        <child link="${namespace}_${name}_infra1_frame" />
       </joint>
-      <link name="${name}_infra1_frame"/>
-      <joint name="${name}_infra1_optical_joint" type="fixed">
+      <link name="${namespace}_${name}_infra1_frame"/>
+      <joint name="${namespace}_${name}_infra1_optical_joint" type="fixed">
         <origin xyz="0 0 0" rpy="${-M_PI/2} 0 ${-M_PI/2}" />
-        <parent link="${name}_infra1_frame" />
-        <child link="${name}_infra1_optical_frame" />
+        <parent link="${namespace}_${name}_infra1_frame" />
+        <child link="${namespace}_${name}_infra1_optical_frame" />
       </joint>
-      <link name="${name}_infra1_optical_frame"/>
+      <link name="${namespace}_${name}_infra1_optical_frame"/>
       <!-- camera right IR joints and links -->
-      <joint name="${name}_infra2_joint" type="fixed">
+      <joint name="${namespace}_${name}_infra2_joint" type="fixed">
         <origin xyz="0 ${d435_cam_depth_to_infra2_offset} 0" rpy="0 0 0" />
-        <parent link="${name}_link" />
-        <child link="${name}_infra2_frame" />
+        <parent link="${namespace}_${name}_link" />
+        <child link="${namespace}_${name}_infra2_frame" />
       </joint>
-      <link name="${name}_infra2_frame"/>
-      <joint name="${name}_infra2_optical_joint" type="fixed">
+      <link name="${namespace}_${name}_infra2_frame"/>
+      <joint name="${namespace}_${name}_infra2_optical_joint" type="fixed">
         <origin xyz="0 0 0" rpy="${-M_PI/2} 0 ${-M_PI/2}" />
-        <parent link="${name}_infra2_frame" />
-        <child link="${name}_infra2_optical_frame" />
+        <parent link="${namespace}_${name}_infra2_frame" />
+        <child link="${namespace}_${name}_infra2_optical_frame" />
       </joint>
-      <link name="${name}_infra2_optical_frame"/>
+      <link name="${namespace}_${name}_infra2_optical_frame"/>
       <!-- camera color joints and links -->
-      <joint name="${name}_color_joint" type="fixed">
+      <joint name="${namespace}_${name}_color_joint" type="fixed">
         <origin xyz="0 ${d435_cam_depth_to_color_offset} 0" rpy="0 0 0" />
-        <parent link="${name}_link" />
-        <child link="${name}_color_frame" />
+        <parent link="${namespace}_${name}_link" />
+        <child link="${namespace}_${name}_color_frame" />
       </joint>
-      <link name="${name}_color_frame"/>
-      <joint name="${name}_color_optical_joint" type="fixed">
+      <link name="${namespace}_${name}_color_frame"/>
+      <joint name="${namespace}_${name}_color_optical_joint" type="fixed">
         <origin xyz="0 0 0" rpy="${-M_PI/2} 0 ${-M_PI/2}" />
-        <parent link="${name}_color_frame" />
-        <child link="${name}_color_optical_frame" />
+        <parent link="${namespace}_${name}_color_frame" />
+        <child link="${namespace}_${name}_color_optical_frame" />
       </joint>
-      <link name="${name}_color_optical_frame"/>
+      <link name="${namespace}_${name}_color_optical_frame"/>
     </xacro:if>
     <xacro:if value="${add_plug}">
-      <xacro:usb_plug parent="${name}_link" name="${name}_usb_plug">
+      <xacro:usb_plug parent="${namespace}_${name}_link" name="${namespace}_${name}_usb_plug">
         <origin xyz="${d435_cam_mount_from_center_offset - 0.02095} ${-d435_cam_depth_py - 0.0353} 0" rpy="0 0 0"/>
       </xacro:usb_plug>
     </xacro:if>
     <!-- gazebo realsense plugin -->
-    <gazebo reference="${name}_link">
-      <sensor name="${name}" type="depth">
+    <gazebo reference="${namespace}_${name}_link">
+      <sensor name="${namespace}_${name}" type="depth">
         <always_on>true</always_on>
         <update_rate>60</update_rate>
         <visualize>false</visualize>
-        <camera name="${name}">
+        <camera name="${namespace}_${name}">
           <horizontal_fov>1.57</horizontal_fov>
           <image>
@@ -170,21 +169,22 @@
           </distortion>
         </camera>
-        <plugin name="camera_plugin" filename="libgazebo_ros_camera.so">
+        <plugin name="${name}_plugin" filename="libgazebo_ros_camera.so">
           <ros>
-            <remapping>camera/image_raw:=camera/color/image_raw</remapping>
-            <remapping>camera/image_raw/compressed:=camera/color/image_raw/compressed</remapping>
-            <remapping>camera/image_raw/compressedDepth:=camera/color/image_raw/compressedDepth</remapping>
-            <remapping>camera/camera_info:=camera/color/camera_info</remapping>
-            <remapping>camera/depth/image_raw:=camera/aligned_depth_to_color/image_raw</remapping>
-            <remapping>camera/depth/image_raw/compressed:=camera/aligned_depth_to_color/image_raw/compressed</remapping>
-            <remapping>camera/depth/image_raw/compressedDepth:=camera/aligned_depth_to_color/image_raw/compressedDepth</remapping>
-            <remapping>camera/depth/camera_info:=camera/aligned_depth_to_color/camera_info</remapping>
-            <remapping>camera/points:=camera/depth/color/points</remapping>
+            <namespace>${namespace}</namespace>
+            <remapping>${name}/image_raw:=${name}/color/image_raw</remapping>
+            <remapping>${name}/image_raw/compressed:=${name}/color/image_raw/compressed</remapping>
+            <remapping>${name}/image_raw/compressedDepth:=${name}/color/image_raw/compressedDepth</remapping>
+            <remapping>${name}/camera_info:=${name}/color/camera_info</remapping>
+            <remapping>${name}/depth/image_raw:=${name}/aligned_depth_to_color/image_raw</remapping>
+            <remapping>${name}/depth/image_raw/compressed:=${name}/aligned_depth_to_color/image_raw/compressed</remapping>
+            <remapping>${name}/depth/image_raw/compressedDepth:=${name}/aligned_depth_to_color/image_raw/compressedDepth</remapping>
+            <remapping>${name}/depth/camera_info:=${name}/aligned_depth_to_color/camera_info</remapping>
+            <remapping>${name}/points:=${name}/depth/color/points</remapping>
           </ros>
           <baseline>0.05</baseline>
           <always_on>true</always_on>
           <update_rate>0.0</update_rate>
-          <frame_name>${name}_color_optical_frame</frame_name>
-          <camera_name>camera</camera_name>
+          <frame_name>${namespace}_${name}_color_optical_frame</frame_name>
+          <camera_name>${name}</camera_name>
           <min_depth>0.3</min_depth>
           <max_depth>3.0</max_depth>

File: vault_description/urdf/sensors/realsense/d435i.urdf.xacro (robot description, xacro)
@@ -9,9 +9,9 @@
   <xacro:include filename="$(find vault_description)/urdf/sensors/realsense/d435.urdf.xacro"/>
   <xacro:include filename="$(find vault_description)/urdf/sensors/realsense/d435i_imu_modules.urdf.xacro"/>
-  <xacro:macro name="sensor_d435i" params="parent *origin name:=camera use_nominal_extrinsics:=false">
-    <xacro:sensor_d435 parent="${parent}" name="${name}" use_nominal_extrinsics="${use_nominal_extrinsics}">
+  <xacro:macro name="sensor_d435i" params="parent *origin name:=d435i namespace:=vault use_nominal_extrinsics:=true add_plug:=false use_mesh:=true">
+    <xacro:sensor_d435 parent="${parent}" name="${name}" namespace="${namespace}" use_nominal_extrinsics="${use_nominal_extrinsics}">
       <xacro:insert_block name="origin" />
     </xacro:sensor_d435>
-    <xacro:d435i_imu_modules name="${name}" use_nominal_extrinsics="${use_nominal_extrinsics}"/>
+    <xacro:d435i_imu_modules name="${name}" namespace="${namespace}" use_nominal_extrinsics="${use_nominal_extrinsics}"/>
   </xacro:macro>
 </robot>

File: vault_description/urdf/sensors/realsense/d435i_imu_modules.urdf.xacro (robot description, xacro)
@@ -7,51 +7,52 @@
 -->
 <robot name="d435i_imu_modules" xmlns:xacro="http://www.ros.org/wiki/xacro">
-  <xacro:macro name="d435i_imu_modules" params="name use_nominal_extrinsics">
+  <xacro:macro name="d435i_imu_modules" params="name:=d435i namespace:=vault use_nominal_extrinsics">
     <xacro:property name="M_PI" value="${pi}" />
     <xacro:if value="${use_nominal_extrinsics}">
-      <link name="${name}_accel_frame" />
-      <link name="${name}_accel_optical_frame" />
-      <link name="${name}_gyro_frame" />
-      <link name="${name}_gyro_optical_frame" />
-      <link name="${name}_imu_frame" />
-      <link name="${name}_imu_optical_frame" />
-      <joint name="${name}_accel_joint" type="fixed">
+      <link name="${namespace}_${name}_accel_frame" />
+      <link name="${namespace}_${name}_accel_optical_frame" />
+      <link name="${namespace}_${name}_gyro_frame" />
+      <link name="${namespace}_${name}_gyro_optical_frame" />
+      <link name="${namespace}_${name}_imu_frame" />
+      <link name="${namespace}_${name}_imu_optical_frame" />
+      <joint name="${namespace}_${name}_accel_joint" type="fixed">
         <origin xyz = "-0.01174 -0.00552 0.0051" rpy = "0 0 0" />
-        <parent link="${name}_link" />
-        <child link="${name}_accel_frame" />
+        <parent link="${namespace}_${name}_link" />
+        <child link="${namespace}_${name}_accel_frame" />
       </joint>
-      <joint name="${name}_accel_optical_joint" type="fixed">
+      <joint name="${namespace}_${name}_accel_optical_joint" type="fixed">
         <origin xyz = "0 0 0" rpy = "${-M_PI/2} 0 ${-M_PI/2}" />
-        <parent link="${name}_accel_frame" />
-        <child link="${name}_accel_optical_frame" />
+        <parent link="${namespace}_${name}_accel_frame" />
+        <child link="${namespace}_${name}_accel_optical_frame" />
       </joint>
-      <joint name="${name}_gyro_joint" type="fixed">
+      <joint name="${namespace}_${name}_gyro_joint" type="fixed">
         <origin xyz = "-0.01174 -0.00552 0.0051" rpy = "0 0 0" />
-        <parent link="${name}_link" />
-        <child link="${name}_gyro_frame" />
+        <parent link="${namespace}_${name}_link" />
+        <child link="${namespace}_${name}_gyro_frame" />
       </joint>
-      <joint name="${name}_gyro_optical_joint" type="fixed">
+      <joint name="${namespace}_${name}_gyro_optical_joint" type="fixed">
         <origin xyz = "0 0 0" rpy = "${-M_PI/2} 0 ${-M_PI/2}" />
-        <parent link="${name}_gyro_frame" />
-        <child link="${name}_gyro_optical_frame" />
+        <parent link="${namespace}_${name}_gyro_frame" />
+        <child link="${namespace}_${name}_gyro_optical_frame" />
       </joint>
-      <joint name="${name}_imu_joint" type="fixed">
+      <joint name="${namespace}_${name}_imu_joint" type="fixed">
         <origin xyz = "-0.01174 -0.00552 0.0051" rpy = "0 0 0" />
-        <parent link="${name}_link" />
-        <child link="${name}_imu_frame" />
+        <parent link="${namespace}_${name}_link" />
+        <child link="${namespace}_${name}_imu_frame" />
       </joint>
-      <joint name="${name}_imu_optical_joint" type="fixed">
+      <joint name="${namespace}_${name}_imu_optical_joint" type="fixed">
         <origin xyz = "0 0 0" rpy = "${-M_PI/2} 0 ${-M_PI/2}" />
-        <parent link="${name}_imu_frame" />
-        <child link="${name}_imu_optical_frame" />
+        <parent link="${namespace}_${name}_imu_frame" />
+        <child link="${namespace}_${name}_imu_optical_frame" />
       </joint>
-      <gazebo reference="${name}_imu_optical_frame">
-        <sensor name="camera_imu_sensor" type="imu">
+      <gazebo reference="${namespace}_${name}_imu_optical_frame">
+        <sensor name="${name}_imu_plugin" type="imu">
           <plugin filename="libgazebo_ros_imu_sensor.so" name="imu_controller">
             <ros>
-              <remapping>~/out:=camera/imu</remapping>
+              <namespace>${namespace}</namespace>
+              <remapping>~/out:=${name}/imu</remapping>
             </ros>
             <initial_orientation_as_reference>false</initial_orientation_as_reference>
-            <frame_name>${name}_imu_optical_frame</frame_name>
+            <frame_name>${namespace}_${name}_imu_optical_frame</frame_name>
           </plugin>
           <always_on>true</always_on>
