Commit message: d435i + t265

File: vault_description/urdf/sensors/realsense/t265.urdf.xacro (robot description, xacro)
@@ -1,7 +1,7 @@
 <?xml version="1.0"?>
 <robot name="sensor_t265" xmlns:xacro="http://ros.org/wiki/xacro">
-    <xacro:macro name="t265_fisheye" params="name reference_frame topic">
-        <gazebo reference="${name}_link">
-            <sensor name="camera" type="wideanglecamera">
+    <xacro:macro name="t265_fisheye" params="name namespace reference_frame topic">
+        <gazebo reference="${namespace}_${name}_link">
+            <sensor name="${name}_${topic}" type="wideanglecamera">
                 <camera>
                     <horizontal_fov>6.283</horizontal_fov>
@@ -36,7 +36,10 @@
                     </distortion>
                 </camera>
-                <plugin name="${topic}_camera_controller" filename="libgazebo_ros_camera.so">
+                <plugin name="${name}_${topic}_plugin" filename="libgazebo_ros_camera.so">
+                    <ros>
+                        <namespace>${namespace}</namespace>
+                    </ros>
                     <always_on>true</always_on>
-                    <camera_name>camera/${topic}</camera_name>
+                    <camera_name>${name}/${topic}</camera_name>
                     <frame_name>${reference_frame}</frame_name>
                     <hack_baseline>-0.0</hack_baseline>
@@ -48,13 +51,13 @@
         </gazebo>
     </xacro:macro>
-    <xacro:macro name="sensor_t265" params="name parent *origin">
+    <xacro:macro name="sensor_t265" params="name:=t265 namespace:=vault parent base_link *origin">
         <xacro:include filename="$(find vault_description)/urdf/sensors/realsense/materials.urdf.xacro" />
         <xacro:property name="M_PI" value="3.1415926535897931" />
-        <joint name="${name}_pose_frame_joint" type="fixed">
+        <joint name="${namespace}_${name}_pose_frame_joint" type="fixed">
             <parent link="${parent}"/>
-            <child link="${name}_pose_frame"/>
+            <child link="${namespace}_${name}_pose_frame"/>
             <xacro:insert_block name="origin"/>
         </joint>
-        <link name="${name}_pose_frame">
+        <link name="${namespace}_${name}_pose_frame">
             <visual>
                 <origin rpy="1.57 0 1.57" xyz="0 0 0"/>
@@ -80,92 +83,94 @@
             </inertial>
         </link>
-        <gazebo reference="${name}_pose_frame">
+        <gazebo reference="${namespace}_${name}_pose_frame">
         <material>Gazebo/Silver</material>
         </gazebo>
-        <joint name="${name}_joint" type="fixed">
-            <parent link="${name}_pose_frame"/>
-            <child link="${name}_link"/>
+        <joint name="${namespace}_${name}_joint" type="fixed">
+            <parent link="${namespace}_${name}_pose_frame"/>
+            <child link="${namespace}_${name}_link"/>
             <origin rpy="0 0 0" xyz="0 0 0"/>
         </joint>
-        <link name="${name}_link"/>
-        <joint name="${name}_fisheye1_joint" type="fixed">
-            <parent link="${name}_link"/>
-            <child link="${name}_fisheye1_frame"/>
+        <link name="${namespace}_${name}_link"/>
+        <joint name="${namespace}_${name}_fisheye1_joint" type="fixed">
+            <parent link="${namespace}_${name}_link"/>
+            <child link="${namespace}_${name}_fisheye1_frame"/>
             <origin rpy="${M_PI} 0 ${M_PI}" xyz="0 0.032 0"/>
         </joint>
-        <link name="${name}_fisheye1_frame"/>
-        <joint name="${name}_ligned_depth_to_fisheye1_joint" type="fixed">
-            <parent link="${name}_link"/>
-            <child link="${name}_aligned_depth_to_fisheye1_frame"/>
+        <link name="${namespace}_${name}_fisheye1_frame"/>
+        <joint name="${namespace}_${name}_ligned_depth_to_fisheye1_joint" type="fixed">
+            <parent link="${namespace}_${name}_link"/>
+            <child link="${namespace}_${name}_aligned_depth_to_fisheye1_frame"/>
             <origin rpy="${M_PI} 0 ${M_PI}" xyz="0 0.032 0"/>
         </joint>
-        <link name="${name}_aligned_depth_to_fisheye1_frame"/>
-        <joint name="${name}_fisheye1_optical_joint" type="fixed">
-            <parent link="${name}_aligned_depth_to_fisheye1_frame"/>
-            <child link="${name}_fisheye1_optical_frame"/>
-            <origin rpy="${M_PI/2} 0 -${M_PI/2}" xyz="0 0 0"/>
-        </joint>
-        <link name="${name}_fisheye1_optical_frame"/>
+        <link name="${namespace}_${name}_aligned_depth_to_fisheye1_frame"/>
+        <joint name="${namespace}_${name}_fisheye1_optical_joint" type="fixed">
+            <parent link="${namespace}_${name}_aligned_depth_to_fisheye1_frame"/>
+            <child link="${namespace}_${name}_fisheye1_optical_frame"/>
+            <origin rpy="${M_PI/2} 0 -${M_PI/2}" xyz="0 0 0"/>
+        </joint>
+        <link name="${namespace}_${name}_fisheye1_optical_frame"/>
         <xacro:t265_fisheye
-        name="${name}"
-        reference_frame="${name}_fisheye1_optical_frame"
-        topic="fisheye1">
+            name="${name}"
+            namespace="${namespace}"
+            reference_frame="${namespace}_${name}_fisheye1_optical_frame"
+            topic="fisheye1">
         </xacro:t265_fisheye>
-        <joint name="${name}_fisheye2_joint" type="fixed">
-            <parent link="${name}_link"/>
-            <child link="${name}_fisheye2_frame"/>
+        <joint name="${namespace}_${name}_fisheye2_joint" type="fixed">
+            <parent link="${namespace}_${name}_link"/>
+            <child link="${namespace}_${name}_fisheye2_frame"/>
             <origin rpy="${M_PI} 0 ${M_PI}" xyz="0 -0.032 0"/>
         </joint>
-        <link name="${name}_fisheye2_frame"/>
-        <joint name="${name}_fisheye2_optical_joint" type="fixed">
-            <parent link="${name}_fisheye2_frame"/>
-            <child link="${name}_fisheye2_optical_frame"/>
-            <origin rpy="${M_PI/2} 0 -${M_PI/2}" xyz="0 0 0"/>
-        </joint>
-        <link name="${name}_fisheye2_optical_frame"/>
+        <link name="${namespace}_${name}_fisheye2_frame"/>
+        <joint name="${namespace}_${name}_fisheye2_optical_joint" type="fixed">
+            <parent link="${namespace}_${name}_fisheye2_frame"/>
+            <child link="${namespace}_${name}_fisheye2_optical_frame"/>
+            <origin rpy="${M_PI/2} 0 -${M_PI/2}" xyz="0 0 0"/>
+        </joint>
+        <link name="${namespace}_${name}_fisheye2_optical_frame"/>
         <xacro:t265_fisheye
-        name="${name}"
-        reference_frame="${name}_fisheye2_optical_frame"
-        topic="fisheye2">
+            name="${name}"
+            namespace="${namespace}"
+            reference_frame="${namespace}_${name}_fisheye2_optical_frame"
+            topic="fisheye2">
         </xacro:t265_fisheye>
-        <joint name="${name}_gyro_joint" type="fixed">
-            <parent link="${name}_link"/>
-            <child link="${name}_gyro_frame"/>
+        <joint name="${namespace}_${name}_gyro_joint" type="fixed">
+            <parent link="${namespace}_${name}_link"/>
+            <child link="${namespace}_${name}_gyro_frame"/>
             <origin rpy="0 0 ${M_PI}" xyz="0 0.021 0"/>
         </joint>
-        <link name="${name}_gyro_frame"/>
-        <joint name="${name}_gyro_optical_joint" type="fixed">
-            <parent link="${name}_gyro_frame"/>
-            <child link="${name}_gyro_optical_frame"/>
-            <origin rpy="${M_PI/2} 0 -${M_PI/2}" xyz="0 0 0"/>
-        </joint>
-        <link name="${name}_gyro_optical_frame"/>
-        <joint name="${name}_accel_joint" type="fixed">
-            <parent link="${name}_link"/>
-            <child link="${name}_accel_frame"/>
+        <link name="${namespace}_${name}_gyro_frame"/>
+        <joint name="${namespace}_${name}_gyro_optical_joint" type="fixed">
+            <parent link="${namespace}_${name}_gyro_frame"/>
+            <child link="${namespace}_${name}_gyro_optical_frame"/>
+            <origin rpy="${M_PI/2} 0 -${M_PI/2}" xyz="0 0 0"/>
+        </joint>
+        <link name="${namespace}_${name}_gyro_optical_frame"/>
+        <joint name="${namespace}_${name}_accel_joint" type="fixed">
+            <parent link="${namespace}_${name}_link"/>
+            <child link="${namespace}_${name}_accel_frame"/>
             <origin rpy="0 0 ${M_PI}" xyz="0 0.021 0"/>
         </joint>
-        <link name="${name}_accel_frame"/>
-        <joint name="${name}_accel_optical_joint" type="fixed">
-            <parent link="${name}_accel_frame"/>
-            <child link="${name}_accel_optical_frame"/>
-            <origin rpy="${M_PI/2} 0 -${M_PI/2}" xyz="0 0 0"/>
-        </joint>
-        <link name="${name}_accel_optical_frame"/>
-        <joint name="${name}_imu_joint" type="fixed">
-            <parent link="${name}_link"/>
-            <child link="${name}_imu_frame"/>
+        <link name="${namespace}_${name}_accel_frame"/>
+        <joint name="${namespace}_${name}_accel_optical_joint" type="fixed">
+            <parent link="${namespace}_${name}_accel_frame"/>
+            <child link="${namespace}_${name}_accel_optical_frame"/>
+            <origin rpy="${M_PI/2} 0 -${M_PI/2}" xyz="0 0 0"/>
+        </joint>
+        <link name="${namespace}_${name}_accel_optical_frame"/>
+        <joint name="${namespace}_${name}_imu_joint" type="fixed">
+            <parent link="${namespace}_${name}_link"/>
+            <child link="${namespace}_${name}_imu_frame"/>
             <origin rpy="0 0 ${M_PI}" xyz="0 0.021 0"/>
         </joint>
-        <link name="${name}_imu_frame"/>
-        <joint name="${name}_imu_optical_joint" type="fixed">
-            <parent link="${name}_imu_frame"/>
-            <child link="${name}_imu_optical_frame"/>
-            <origin rpy="${M_PI/2} 0 -${M_PI/2}" xyz="0 0 0"/>
-        </joint>
-        <link name="${name}_imu_optical_frame"/>
-        <gazebo reference="${name}_imu_optical_frame">
+        <link name="${namespace}_${name}_imu_frame"/>
+        <joint name="${namespace}_${name}_imu_optical_joint" type="fixed">
+            <parent link="${namespace}_${name}_imu_frame"/>
+            <child link="${namespace}_${name}_imu_optical_frame"/>
+            <origin rpy="${M_PI/2} 0 -${M_PI/2}" xyz="0 0 0"/>
+        </joint>
+        <link name="${namespace}_${name}_imu_optical_frame"/>
+        <gazebo reference="${namespace}_${name}_imu_optical_frame">
             <gravity>true</gravity>
-            <sensor name="${name}_imu" type="imu">
+            <sensor name="${name}_imu_plugin" type="imu">
                 <always_on>true</always_on>
                 <update_rate>200</update_rate>
@@ -173,7 +178,8 @@
                 <plugin filename="libgazebo_ros_imu_sensor.so" name="imu_plugin">
                     <ros>
-                        <remapping>~/out:=camera/imu</remapping>
+                        <namespace>${namespace}</namespace>
+                        <remapping>~/out:=${name}/imu</remapping>
                     </ros>
-                    <frame_name>${name}_imu_optical_frame</frame_name>
+                    <frame_name>${namespace}_${name}_imu_optical_frame</frame_name>
                 </plugin>
                 <imu>
@@ -235,10 +241,11 @@
         <!-- odom -->
         <gazebo>
-            <plugin name="p3d_base_controller" filename="libgazebo_ros_p3d.so">
+            <plugin name="${name}_p3d_plugin" filename="libgazebo_ros_p3d.so">
                 <ros>
-                    <remapping>odom:=camera/pose/sample</remapping>
+                    <namespace>${namespace}</namespace>
+                    <remapping>odom:=${name}/pose/sample</remapping>
                 </ros>
                 <always_on>true</always_on>
-                <body_name>base_link</body_name>
+                <body_name>${base_link}</body_name>
                 <frame_name>odom</frame_name>
                 <update_rate>200</update_rate>

File: vault_description/urdf/vault.urdf.xacro (robot description, xacro)
@@ -2,5 +2,4 @@
 <robot name="vault" xmlns:xacro="http://www.ros.org/wiki/xacro">
     <xacro:macro name="vault" params="parent *origin">
-        <xacro:arg name="t265" default="false"/>
         <!-- Include macros -->
         <xacro:include filename="$(find vault_description)/urdf/inertials.xacro"/>
@@ -38,22 +37,17 @@
         <xacro:vault_battery parent="vault_box_link" />
         <!-- sensors -->
-        <xacro:unless value="$(arg t265)">
-            <xacro:arg name="use_nominal_extrinsics" default="true" />
-            <xacro:sensor_d435i parent="vault_realsense_mount_link" name="vault_camera" use_nominal_extrinsics="$(arg use_nominal_extrinsics)">
-                <origin xyz="0 -0.005 -0.0075" rpy="0 0 -1.57"/>
-            </xacro:sensor_d435i>
-        </xacro:unless>
-        <xacro:if value="$(arg t265)">
-            <xacro:sensor_t265 name="vault_camera" parent="vault_realsense_mount_link">
-                <origin xyz="0 -0.01 0.0075" rpy="0 0 -1.57"/>
-            </xacro:sensor_t265>
-        </xacro:if>
-        <xacro:sensor_imu name="vault_imu" parent="vault_box_link">
+        <xacro:sensor_d435i parent="vault_realsense_mount_link" name="d435i" namespace="vault">
+            <origin xyz="0 -0.005 -0.0075" rpy="0 0 -1.57"/>
+        </xacro:sensor_d435i>
+        <xacro:sensor_t265 parent="vault_realsense_mount_link" name="t265" namespace="vault" base_link="${parent}">
+            <origin xyz="-0.01 0.0035 0.035" rpy="0 0 -1.57"/>
+        </xacro:sensor_t265>
+        <xacro:sensor_imu name="imu" namespace="vault" parent="vault_box_link">
             <origin xyz="0 -0.075 0.084" rpy="0 -3.141516 0"/>
         </xacro:sensor_imu>
-        <xacro:sensor_gps name="vault_gps" parent="vault_box_link">
+        <xacro:sensor_gps name="gps" namespace="vault" parent="vault_box_link">
             <origin xyz="0 0 0.1075" rpy="0 0 0"/>
         </xacro:sensor_gps>
-        <xacro:gps_board name="vault_gps" parent="vault_box_link">
+        <xacro:gps_board name="gps" namespace="vault" parent="vault_box_link">
             <origin xyz="-0.077 0 -0.010" rpy="0 1.57 0"/>
         </xacro:gps_board>
