Commit message: new box models

File: vault_description/urdf/box/battery.urdf.xacro (robot description, xacro)
@@ -2,7 +2,7 @@
 <robot name="vault_battery" xmlns:xacro="http://www.ros.org/wiki/xacro">
     <xacro:macro name="vault_battery" params="parent">
-        <xacro:property name="box_heigh" value="0.076" />
+        <xacro:property name="box_heigh" value="0.038" />
         <xacro:property name="box_width" value="0.158" />
-        <xacro:property name="box_depth" value="0.038" />
+        <xacro:property name="box_depth" value="0.076" />
         <xacro:property name="box_mass" value="1.000" />
         <link name="vault_battery_link">
@@ -29,5 +29,5 @@
         </gazebo>
         <joint name="vault_battery_joint" type="fixed">
-            <origin rpy="0 0 0" xyz="0 0.08 -0.002"/>
+            <origin rpy="0 0 0" xyz="0 0 0.053"/>
             <parent link="${parent}" />
             <child link="vault_battery_link" />

File: vault_description/urdf/box/box.urdf.xacro (robot description, xacro)
@@ -2,11 +2,11 @@
 <robot name="vault_box" xmlns:xacro="http://www.ros.org/wiki/xacro">
     <xacro:macro name="vault_box" params="parent">
-        <xacro:property name="box_heigh" value="0.120" />
+        <xacro:property name="box_heigh" value="0.150" />
         <xacro:property name="box_width" value="0.190" />
-        <xacro:property name="box_depth" value="0.210" />
-        <xacro:property name="box_mass" value="0.25" />
+        <xacro:property name="box_depth" value="0.190" />
+        <xacro:property name="box_mass" value="0.2" />
         <link name="vault_box_link">
             <visual>
-                <origin rpy="0 0 0" xyz="0 0 -0.06" />
+                <origin rpy="0 0 0" xyz="0 0 -0.075" />
                 <geometry>
                     <mesh filename="package://vault_description/meshes/box/box.stl" scale="0.001 0.001 0.001"/>

File: vault_description/urdf/box/computer.urdf.xacro (robot description, xacro)
@@ -12,5 +12,5 @@
                     <box size="${box_width} ${box_depth} ${box_heigh}"/>
                 </geometry>
-                <material name="dark_gray" />
+                <material name="white" />
             </visual>
             <collision>
@@ -26,8 +26,8 @@
         </link>
         <gazebo reference="vault_computer_link">
-            <material>Gazebo/DarkGrey</material>
+            <material>Gazebo/White</material>
         </gazebo>
         <joint name="vault_computer_joint" type="fixed">
-            <origin rpy="0 0 0" xyz="0 0 0.060"/>
+            <origin rpy="0 0 0" xyz="0 0 0.014"/>
             <parent link="${parent}" />
             <child link="vault_computer_link" />

File: vault_description/urdf/box/cover.urdf.xacro (robot description, xacro)
@@ -2,13 +2,13 @@
 <robot name="vault_cover" xmlns:xacro="http://www.ros.org/wiki/xacro">
     <xacro:macro name="vault_cover" params="parent">
-        <xacro:property name="box_heigh" value="0.0085" />
-        <xacro:property name="box_width" value="0.168" />
-        <xacro:property name="box_depth" value="0.213" />
+        <xacro:property name="box_heigh" value="0.003" />
+        <xacro:property name="box_width" value="0.186" />
+        <xacro:property name="box_depth" value="0.194" />
         <xacro:property name="box_mass" value="0.01" />
         <link name="vault_cover_link">
             <visual>
-                <origin rpy="0 0 0" xyz="0 -0.008 -0.015" />
+                <origin rpy="0 0 0" xyz="0 0 0" />
                 <geometry>
-                    <mesh filename="package://vault_description/meshes/box/cover.stl" scale="0.001 0.001 0.001"/>
+                    <box size="${box_width} ${box_depth} ${box_heigh}"/>
                 </geometry>
                 <material name="red" />
@@ -29,5 +29,5 @@
         </gazebo>
         <joint name="vault_cover_joint" type="fixed">
-            <origin rpy="0 0 0" xyz="0 0.006 -0.0445"/>
+            <origin rpy="0 0 0" xyz="-0.004 -0.005 -0.0725"/>
             <parent link="${parent}" />
             <child link="vault_cover_link" />

File: vault_description/urdf/box/realsense_mount.urdf.xacro (robot description, xacro)
@@ -4,9 +4,9 @@
         <xacro:property name="box_heigh" value="0.033" />
         <xacro:property name="box_width" value="0.080" />
-        <xacro:property name="box_depth" value="0.030" />
+        <xacro:property name="box_depth" value="0.040" />
         <xacro:property name="box_mass" value="0.1" />
         <link name="vault_realsense_mount_link">
             <visual>
-                <origin rpy="0 0 0" xyz="0.002 0.069 -0.0675" />
+                <origin rpy="0 0 0" xyz="0.002 0.0715 -0.075" />
                 <geometry>
                     <mesh filename="package://vault_description/meshes/box/realsense_mount.stl"  scale="0.001 0.001 0.001"/>
@@ -29,5 +29,5 @@
         </gazebo>
         <joint name="vault_realsense_mount_joint" type="fixed">
-            <origin rpy="0 0 0" xyz="0 -0.0695 0.0075"/>
+            <origin rpy="0 0 0" xyz="0 -0.072 0"/>
             <parent link="${parent}" />
             <child link="vault_realsense_mount_link" />

File: vault_description/urdf/vault.urdf.xacro (robot description, xacro)
@@ -39,14 +39,14 @@
         <xacro:arg name="use_nominal_extrinsics" default="true" />
         <xacro:sensor_d435i parent="vault_realsense_mount_link" name="vault_camera" use_nominal_extrinsics="$(arg use_nominal_extrinsics)">
-            <origin xyz="0 -0.005 -0.005" rpy="0 0 -1.57"/>
+            <origin xyz="0 -0.005 -0.0075" rpy="0 0 -1.57"/>
         </xacro:sensor_d435i>
         <xacro:sensor_imu name="vault_imu" parent="vault_box_link">
-            <origin xyz="0.075 -0.05 0" rpy="0 -1.57 0"/>
+            <origin xyz="0.083 -0.060 0" rpy="0 -1.57 0"/>
         </xacro:sensor_imu>
         <xacro:sensor_gps name="vault_gps" parent="vault_box_link">
-            <origin xyz="0 0 0.1025" rpy="0 0 0"/>
+            <origin xyz="0 0 0.0865" rpy="0 0 0"/>
         </xacro:sensor_gps>
         <xacro:gps_board name="vault_gps" parent="vault_box_link">
-            <origin xyz="-0.072 -0.005 0" rpy="0 1.57 0"/>
+            <origin xyz="-0.079 -0.005 0" rpy="0 1.57 0"/>
         </xacro:gps_board>
     </xacro:macro>

Commit message: new models

File: vault_description/urdf/box/battery.urdf.xacro (robot description, xacro)
@@ -29,5 +29,5 @@
         </gazebo>
         <joint name="vault_battery_joint" type="fixed">
-            <origin rpy="0 0 0" xyz="0 0 0.053"/>
+            <origin rpy="0 0 0" xyz="0 0 0.073"/>
             <parent link="${parent}" />
             <child link="vault_battery_link" />

File: vault_description/urdf/box/box.urdf.xacro (robot description, xacro)
@@ -2,11 +2,11 @@
 <robot name="vault_box" xmlns:xacro="http://www.ros.org/wiki/xacro">
     <xacro:macro name="vault_box" params="parent">
-        <xacro:property name="box_heigh" value="0.150" />
+        <xacro:property name="box_heigh" value="0.190" />
         <xacro:property name="box_width" value="0.190" />
         <xacro:property name="box_depth" value="0.190" />
-        <xacro:property name="box_mass" value="0.2" />
+        <xacro:property name="box_mass" value="0.1" />
         <link name="vault_box_link">
             <visual>
-                <origin rpy="0 0 0" xyz="0 0 -0.075" />
+                <origin rpy="0 0 0" xyz="0 0 -0.095" />
                 <geometry>
                     <mesh filename="package://vault_description/meshes/box/box.stl" scale="0.001 0.001 0.001"/>

File: vault_description/urdf/box/computer.urdf.xacro (robot description, xacro)
@@ -29,5 +29,5 @@
         </gazebo>
         <joint name="vault_computer_joint" type="fixed">
-            <origin rpy="0 0 0" xyz="0 0 0.014"/>
+            <origin rpy="0 0 0" xyz="0 0 0.034"/>
             <parent link="${parent}" />
             <child link="vault_computer_link" />

File: vault_description/urdf/box/cover.urdf.xacro (robot description, xacro)
@@ -3,6 +3,6 @@
     <xacro:macro name="vault_cover" params="parent">
         <xacro:property name="box_heigh" value="0.003" />
-        <xacro:property name="box_width" value="0.186" />
-        <xacro:property name="box_depth" value="0.194" />
+        <xacro:property name="box_width" value="0.180" />
+        <xacro:property name="box_depth" value="0.200" />
         <xacro:property name="box_mass" value="0.01" />
         <link name="vault_cover_link">
@@ -29,5 +29,5 @@
         </gazebo>
         <joint name="vault_cover_joint" type="fixed">
-            <origin rpy="0 0 0" xyz="-0.004 -0.005 -0.0725"/>
+            <origin rpy="0 0 0" xyz="-0.005 -0.005 -0.0895"/>
             <parent link="${parent}" />
             <child link="vault_cover_link" />

File: vault_description/urdf/box/realsense_mount.urdf.xacro (robot description, xacro)
@@ -8,5 +8,5 @@
         <link name="vault_realsense_mount_link">
             <visual>
-                <origin rpy="0 0 0" xyz="0.002 0.0715 -0.075" />
+                <origin rpy="0 0 0" xyz="0.060 0.080 -0.0165" />
                 <geometry>
                     <mesh filename="package://vault_description/meshes/box/realsense_mount.stl"  scale="0.001 0.001 0.001"/>
@@ -29,5 +29,5 @@
         </gazebo>
         <joint name="vault_realsense_mount_joint" type="fixed">
-            <origin rpy="0 0 0" xyz="0 -0.072 0"/>
+            <origin rpy="0 0 0" xyz="0 -0.077 -0.0075"/>
             <parent link="${parent}" />
             <child link="vault_realsense_mount_link" />

File: vault_description/urdf/vault.urdf.xacro (robot description, xacro)
@@ -42,11 +42,11 @@
         </xacro:sensor_d435i>
         <xacro:sensor_imu name="vault_imu" parent="vault_box_link">
-            <origin xyz="0.083 -0.060 0" rpy="0 -1.57 0"/>
+            <origin xyz="0.079 -0.060 0" rpy="0 -1.57 0"/>
         </xacro:sensor_imu>
         <xacro:sensor_gps name="vault_gps" parent="vault_box_link">
-            <origin xyz="0 0 0.0865" rpy="0 0 0"/>
+            <origin xyz="0 0 0.1015" rpy="0 0 0"/>
         </xacro:sensor_gps>
         <xacro:gps_board name="vault_gps" parent="vault_box_link">
-            <origin xyz="-0.079 -0.005 0" rpy="0 1.57 0"/>
+            <origin xyz="-0.079 -0.005 -0.010" rpy="0 1.57 0"/>
         </xacro:gps_board>
     </xacro:macro>

Commit message: description fixed

File: vault_description/urdf/box/battery.urdf.xacro (robot description, xacro)
@@ -29,5 +29,5 @@
         </gazebo>
         <joint name="vault_battery_joint" type="fixed">
-            <origin rpy="0 0 0" xyz="0 0 0.073"/>
+            <origin rpy="0 0 0" xyz="0 0.054 0.073"/>
             <parent link="${parent}" />
             <child link="vault_battery_link" />

File: vault_description/urdf/box/box.urdf.xacro (robot description, xacro)
@@ -8,5 +8,5 @@
         <link name="vault_box_link">
             <visual>
-                <origin rpy="0 0 0" xyz="0 0 -0.095" />
+                <origin rpy="0 0 0" xyz="0.005 0.005 -0.095" />
                 <geometry>
                     <mesh filename="package://vault_description/meshes/box/box.stl" scale="0.001 0.001 0.001"/>

File: vault_description/urdf/box/computer.urdf.xacro (robot description, xacro)
@@ -29,5 +29,5 @@
         </gazebo>
         <joint name="vault_computer_joint" type="fixed">
-            <origin rpy="0 0 0" xyz="0 0 0.034"/>
+            <origin rpy="0 0 0" xyz="0 0.037 0.034"/>
             <parent link="${parent}" />
             <child link="vault_computer_link" />

File: vault_description/urdf/box/cover.urdf.xacro (robot description, xacro)
@@ -29,5 +29,5 @@
         </gazebo>
         <joint name="vault_cover_joint" type="fixed">
-            <origin rpy="0 0 0" xyz="-0.005 -0.005 -0.0895"/>
+            <origin rpy="0 0 0" xyz="0 0 -0.0895"/>
             <parent link="${parent}" />
             <child link="vault_cover_link" />

File: vault_description/urdf/box/realsense_mount.urdf.xacro (robot description, xacro)
@@ -29,5 +29,5 @@
         </gazebo>
         <joint name="vault_realsense_mount_joint" type="fixed">
-            <origin rpy="0 0 0" xyz="0 -0.077 -0.0075"/>
+            <origin rpy="0 0 0" xyz="0 -0.072 -0.0075"/>
             <parent link="${parent}" />
             <child link="vault_realsense_mount_link" />

File: vault_description/urdf/vault.urdf.xacro (robot description, xacro)
@@ -42,11 +42,11 @@
         </xacro:sensor_d435i>
         <xacro:sensor_imu name="vault_imu" parent="vault_box_link">
-            <origin xyz="0.079 -0.060 0" rpy="0 -1.57 0"/>
+            <origin xyz="0 -0.075 0.084" rpy="0 -3.141516 0"/>
         </xacro:sensor_imu>
         <xacro:sensor_gps name="vault_gps" parent="vault_box_link">
-            <origin xyz="0 0 0.1015" rpy="0 0 0"/>
+            <origin xyz="0 0 0.1075" rpy="0 0 0"/>
         </xacro:sensor_gps>
         <xacro:gps_board name="vault_gps" parent="vault_box_link">
-            <origin xyz="-0.079 -0.005 -0.010" rpy="0 1.57 0"/>
+            <origin xyz="-0.077 0 -0.010" rpy="0 1.57 0"/>
         </xacro:gps_board>
     </xacro:macro>

Commit message: description fixed

File: vault_description/urdf/box/battery.urdf.xacro (robot description, xacro)
@@ -2,7 +2,7 @@
 <robot name="vault_battery" xmlns:xacro="http://www.ros.org/wiki/xacro">
     <xacro:macro name="vault_battery" params="parent">
-        <xacro:property name="box_heigh" value="0.038" />
+        <xacro:property name="box_heigh" value="0.076" />
         <xacro:property name="box_width" value="0.158" />
-        <xacro:property name="box_depth" value="0.076" />
+        <xacro:property name="box_depth" value="0.038" />
         <xacro:property name="box_mass" value="1.000" />
         <link name="vault_battery_link">
@@ -29,5 +29,5 @@
         </gazebo>
         <joint name="vault_battery_joint" type="fixed">
-            <origin rpy="0 0 0" xyz="0 0.054 0.073"/>
+            <origin rpy="0 0 0" xyz="0 0.073 0.014"/>
             <parent link="${parent}" />
             <child link="vault_battery_link" />

File: vault_description/urdf/box/computer.urdf.xacro (robot description, xacro)
@@ -29,5 +29,5 @@
         </gazebo>
         <joint name="vault_computer_joint" type="fixed">
-            <origin rpy="0 0 0" xyz="0 0.037 0.034"/>
+            <origin rpy="0 0 0" xyz="0 0.037 0.072"/>
             <parent link="${parent}" />
             <child link="vault_computer_link" />

File: vault_description/urdf/vault.urdf.xacro (robot description, xacro)
@@ -41,5 +41,5 @@
         </xacro:sensor_d435i>
         <xacro:sensor_t265 parent="vault_realsense_mount_link" name="t265" namespace="vault" base_link="${parent}">
-            <origin xyz="-0.01 0.0035 0.035" rpy="0 0 -1.57"/>
+            <origin xyz="0 0.0035 0.035" rpy="0 0 -1.57"/>
         </xacro:sensor_t265>
         <xacro:sensor_imu name="imu" namespace="vault" parent="vault_box_link">
@@ -50,5 +50,5 @@
         </xacro:sensor_gps>
         <xacro:gps_board name="gps" namespace="vault" parent="vault_box_link">
-            <origin xyz="-0.077 0 -0.010" rpy="0 1.57 0"/>
+            <origin xyz="-0.077 0 -0.010" rpy="1.57 0 1.57"/>
         </xacro:gps_board>
     </xacro:macro>
