Commit message: new description

File: vault_description/urdf/box/computer.urdf.xacro (robot description, xacro)
@@ -29,5 +29,5 @@
         </gazebo>
         <joint name="vault_computer_joint" type="fixed">
-            <origin rpy="0 0 0" xyz="0 0.037 0.072"/>
+            <origin rpy="0 0 0.785" xyz="0 0 0.072"/>
             <parent link="${parent}" />
             <child link="vault_computer_link" />

File: vault_description/urdf/vault.urdf.xacro (robot description, xacro)
@@ -45,5 +45,5 @@
         </xacro:sensor_t265>
         <xacro:sensor_imu name="imu" namespace="vault" parent="vault_box_link">
-            <origin xyz="0 -0.075 0.084" rpy="0 -${M_PI} ${M_PI/2}"/>
+            <origin xyz="0 0 0.044" rpy="0 -${M_PI} ${M_PI/2}"/>
         </xacro:sensor_imu>
         <xacro:sensor_gps name="gps" namespace="vault" parent="vault_box_link">
