Commit message: t265 description fixed

File: vault_description/urdf/sensors/realsense/t265.urdf.xacro (robot description, xacro)
@@ -47,15 +47,10 @@
     <xacro:macro name="sensor_t265" params="name parent rate *origin">
         <xacro:include filename="$(find vault_description)/urdf/sensors/realsense/materials.urdf.xacro" />
-        <joint name="${name}_odom_frame_joint" type="fixed">
+        <xacro:property name="M_PI" value="3.1415926535897931" />
+        <joint name="${name}_pose_frame_joint" type="fixed">
             <parent link="${parent}"/>
-            <child link="${name}_odom_frame"/>
+            <child link="${name}_pose_frame"/>
             <xacro:insert_block name="origin"/>
         </joint>
-        <joint name="${name}_pose_frame_joint" type="fixed">
-            <parent link="${name}_odom_frame"/>
-            <child link="${name}_pose_frame"/>
-            <origin rpy="0 0 0" xyz="0 0 0"/>
-        </joint>
-        <link name="${name}_odom_frame"/>
         <link name="${name}_pose_frame">
             <visual>
@@ -97,6 +92,12 @@
         </joint>
         <link name="${name}_fisheye1_frame"/>
+        <joint name="${name}_ligned_depth_to_fisheye1_joint" type="fixed">
+            <parent link="${name}_link"/>
+            <child link="${name}_aligned_depth_to_fisheye1_frame"/>
+            <origin rpy="0 0 0" xyz="0 0.042 0"/>
+        </joint>
+        <link name="${name}_aligned_depth_to_fisheye1_frame"/>
         <joint name="${name}_fisheye1_optical_joint" type="fixed">
-            <parent link="${name}_fisheye1_frame"/>
+            <parent link="${name}_aligned_depth_to_fisheye1_frame"/>
             <child link="${name}_fisheye1_optical_frame"/>
             <origin rpy="0 0 0" xyz="0.01 0 0"/>
@@ -130,7 +131,13 @@
             <parent link="${name}_link"/>
             <child link="${name}_gyro_frame"/>
-            <origin rpy="0 0 0" xyz="0 0 0"/>
+            <origin rpy="-${M_PI} 0 -${M_PI}" xyz="0 0.02 0"/>
         </joint>
         <link name="${name}_gyro_frame"/>
+        <joint name="${name}_gyro_optical_joint" type="fixed">
+            <parent link="${name}_gyro_frame"/>
+            <child link="${name}_gyro_optical_frame"/>
+            <origin rpy="-${M_PI/2} -${M_PI/2} 0" xyz="0 0 0"/>
+        </joint>
+        <link name="${name}_gyro_optical_frame"/>
         <gazebo reference="${name}_gyro_frame">
             <gravity>true</gravity>
@@ -204,15 +211,21 @@
             <parent link="${name}_link"/>
             <child link="${name}_accel_frame"/>
-            <origin rpy="0 0 0" xyz="0 0 0"/>
+            <origin rpy="0 0 0" xyz="0 0.02 0"/>
         </joint>
         <link name="${name}_accel_frame"/>
+        <joint name="${name}_accel_optical_joint" type="fixed">
+            <parent link="${name}_accel_frame"/>
+            <child link="${name}_accel_optical_frame"/>
+            <origin rpy="-${M_PI/2} -${M_PI/2} 0" xyz="0 0 0"/>
+        </joint>
+        <link name="${name}_accel_optical_frame"/>
         <gazebo>
             <plugin name="p3d_base_controller" filename="libgazebo_ros_p3d.so">
                 <ros>
-                    <remapping>~/out:=${name}/odom/sample</remapping>
+                    <remapping>~/out:=${name}/pose/sample</remapping>
                 </ros>
                 <always_on>true</always_on>
                 <update_rate>${rate}</update_rate>
-                <frame_name>${name}_odom_frame</frame_name>
+                <frame_name>${name}_pose_frame</frame_name>
             </plugin>
         </gazebo>

File: vault_description/urdf/vault.urdf.xacro (robot description, xacro)
@@ -37,11 +37,11 @@
         <xacro:vault_battery parent="vault_box_link" />
         <!-- sensors -->
-        <xacro:arg name="use_nominal_extrinsics" default="true" />
+        <!-- <xacro:arg name="use_nominal_extrinsics" default="true" />
         <xacro:sensor_d435i parent="vault_realsense_mount_link" name="vault_camera" use_nominal_extrinsics="$(arg use_nominal_extrinsics)">
             <origin xyz="0 -0.005 -0.0075" rpy="0 0 -1.57"/>
-        </xacro:sensor_d435i>
-        <!-- <xacro:sensor_t265 name="vault_camera" parent="vault_realsense_mount_link" rate="30">
+        </xacro:sensor_d435i> -->
+        <xacro:sensor_t265 name="vault_camera" parent="vault_realsense_mount_link" rate="30">
             <origin xyz="0 -0.01 0.0075" rpy="0 0 -1.57"/>
-        </xacro:sensor_t265> -->
+        </xacro:sensor_t265>
         <xacro:sensor_imu name="vault_imu" parent="vault_box_link">
             <origin xyz="0 -0.075 0.084" rpy="0 -3.141516 0"/>

Commit message: minor fix

File: vault_description/urdf/sensors/realsense/t265.urdf.xacro (robot description, xacro)
@@ -1,5 +1,5 @@
 <?xml version="1.0"?>
 <robot name="sensor_t265" xmlns:xacro="http://ros.org/wiki/xacro">
-    <xacro:macro name="t265_fisheye" params="name reference_frame topic rate">
+    <xacro:macro name="t265_fisheye" params="name reference_frame topic">
         <gazebo reference="${reference_frame}">
             <sensor name="camera" type="wideanglecamera">
@@ -27,5 +27,5 @@
                     </lens>
                     <always_on>true</always_on>
-                    <update_rate>${rate}</update_rate>
+                    <update_rate>30</update_rate>
                     <distortion>
                         <k1>-0.007419134024530649</k1>
@@ -38,5 +38,5 @@
                 <plugin name="camera_controller" filename="libgazebo_ros_camera.so">
                     <always_on>true</always_on>
-                    <camera_name>${name}/${topic}</camera_name>
+                    <camera_name>camera/${topic}</camera_name>
                     <frame_name>${reference_frame}</frame_name>
                     <hack_baseline>0.07</hack_baseline>
@@ -45,5 +45,5 @@
         </gazebo>
     </xacro:macro>
-    <xacro:macro name="sensor_t265" params="name parent rate *origin">
+    <xacro:macro name="sensor_t265" params="name parent *origin">
         <xacro:include filename="$(find vault_description)/urdf/sensors/realsense/materials.urdf.xacro" />
         <xacro:property name="M_PI" value="3.1415926535897931" />
@@ -107,6 +107,5 @@
         name="${name}"
         reference_frame="${name}_fisheye1_optical_frame"
-        topic="fisheye1"
-        rate="${rate}">
+        topic="fisheye1">
         </xacro:t265_fisheye>
         <joint name="${name}_fisheye2_joint" type="fixed">
@@ -125,6 +124,5 @@
         name="${name}"
         reference_frame="${name}_fisheye2_optical_frame"
-        topic="fisheye2"
-        rate="${rate}">
+        topic="fisheye2">
         </xacro:t265_fisheye>
         <joint name="${name}_gyro_joint" type="fixed">
@@ -144,9 +142,9 @@
             <sensor name="${name}_imu" type="imu">
                 <always_on>true</always_on>
-                <update_rate>${rate}</update_rate>
+                <update_rate>200</update_rate>
                 <visualize>false</visualize>
                 <plugin filename="libgazebo_ros_imu_sensor.so" name="imu_plugin">
                     <ros>
-                        <remapping>~/out:=${name}/gyro/sample</remapping>
+                        <remapping>~/out:=camera/imu</remapping>
                     </ros>
                     <frame_name>${name}_link</frame_name>
@@ -220,12 +218,22 @@
         </joint>
         <link name="${name}_accel_optical_frame"/>
+        <!-- odom -->
+        <!-- <link name="odom"/>
+        <joint name="odom_joint" type="fixed">
+            <parent link="odom"/>
+            <child link="base_link"/>
+            <origin rpy="0 0 0" xyz="0 0 0"/>
+        </joint> -->
         <gazebo>
             <plugin name="p3d_base_controller" filename="libgazebo_ros_p3d.so">
                 <ros>
-                    <remapping>~/out:=${name}/pose/sample</remapping>
+                    <remapping>odom:=odom</remapping>
                 </ros>
-                <always_on>true</always_on>
-                <update_rate>${rate}</update_rate>
-                <frame_name>${name}_pose_frame</frame_name>
+                <body_name>base_link</body_name>
+                <frame_name>odom</frame_name>
+                <update_rate>0</update_rate>
+                <xyz_offset>0 0 0</xyz_offset>
+                <rpy_offset>0 0 0</rpy_offset>
+                <gaussian_noise>0</gaussian_noise>
             </plugin>
         </gazebo>

File: vault_description/urdf/vault.urdf.xacro (robot description, xacro)
@@ -45,5 +45,5 @@
         </xacro:unless>
         <xacro:if value="$(arg t265)">
-            <xacro:sensor_t265 name="vault_camera" parent="vault_realsense_mount_link" rate="30">
+            <xacro:sensor_t265 name="vault_camera" parent="vault_realsense_mount_link">
                 <origin xyz="0 -0.01 0.0075" rpy="0 0 -1.57"/>
             </xacro:sensor_t265>

Commit message: t265 decription fix

File: vault_description/urdf/sensors/realsense/t265.urdf.xacro (robot description, xacro)
@@ -23,5 +23,5 @@
                         </custom_function>
                         <scale_to_hfov>true</scale_to_hfov>
-                        <cutoff_angle>3.1415</cutoff_angle>
+                        <cutoff_angle>${M_PI}</cutoff_angle>
                         <env_texture_size>512</env_texture_size>
                     </lens>
@@ -31,14 +31,17 @@
                         <k1>-0.007419134024530649</k1>
                         <k2>0.041209351271390915</k2>
-                        <k3>-0.03811917081475258</k3>
-                        <p1>0.006366158835589886</p1>
-                        <p2>0.0</p2>
+                        <p1>-0.03811917081475258</p1>
+                        <p2>0.006366158835589886</p2>
+                        <k3>0.0</k3>
                     </distortion>
                 </camera>
-                <plugin name="camera_controller" filename="libgazebo_ros_camera.so">
+                <plugin name="${topic}_camera_controller" filename="libgazebo_ros_camera.so">
                     <always_on>true</always_on>
                     <camera_name>camera/${topic}</camera_name>
                     <frame_name>${reference_frame}</frame_name>
-                    <hack_baseline>0.07</hack_baseline>
+                    <hack_baseline>0.0</hack_baseline>
+                    <focal_length>285.5480041503906</focal_length>
+                    <cx>416.00531005859375</cx>
+                    <cy>403.38909912109375</cy>
                 </plugin>
             </sensor>
@@ -219,18 +222,13 @@
         <link name="${name}_accel_optical_frame"/>
         <!-- odom -->
-        <!-- <link name="odom"/>
-        <joint name="odom_joint" type="fixed">
-            <parent link="odom"/>
-            <child link="base_link"/>
-            <origin rpy="0 0 0" xyz="0 0 0"/>
-        </joint> -->
         <gazebo>
             <plugin name="p3d_base_controller" filename="libgazebo_ros_p3d.so">
                 <ros>
-                    <remapping>odom:=odom</remapping>
+                    <remapping>odom:=camera/pose/sample</remapping>
                 </ros>
+                <always_on>true</always_on>
                 <body_name>base_link</body_name>
                 <frame_name>odom</frame_name>
-                <update_rate>0</update_rate>
+                <update_rate>200</update_rate>
                 <xyz_offset>0 0 0</xyz_offset>
                 <rpy_offset>0 0 0</rpy_offset>

Commit message: t265 description fixed

File: vault_description/urdf/sensors/realsense/t265.urdf.xacro (robot description, xacro)
@@ -2,5 +2,5 @@
 <robot name="sensor_t265" xmlns:xacro="http://ros.org/wiki/xacro">
     <xacro:macro name="t265_fisheye" params="name reference_frame topic">
-        <gazebo reference="${reference_frame}">
+        <gazebo reference="${name}_link">
             <sensor name="camera" type="wideanglecamera">
                 <camera>
@@ -40,5 +40,5 @@
                     <camera_name>camera/${topic}</camera_name>
                     <frame_name>${reference_frame}</frame_name>
-                    <hack_baseline>0.0</hack_baseline>
+                    <hack_baseline>-0.0</hack_baseline>
                     <focal_length>285.5480041503906</focal_length>
                     <cx>416.00531005859375</cx>
@@ -92,5 +92,5 @@
             <parent link="${name}_link"/>
             <child link="${name}_fisheye1_frame"/>
-            <origin rpy="0 0 0" xyz="0 0.042 0"/>
+            <origin rpy="${M_PI} 0 ${M_PI}" xyz="0 0.032 0"/>
         </joint>
         <link name="${name}_fisheye1_frame"/>
@@ -98,5 +98,5 @@
             <parent link="${name}_link"/>
             <child link="${name}_aligned_depth_to_fisheye1_frame"/>
-            <origin rpy="0 0 0" xyz="0 0.042 0"/>
+            <origin rpy="${M_PI} 0 ${M_PI}" xyz="0 0.032 0"/>
         </joint>
         <link name="${name}_aligned_depth_to_fisheye1_frame"/>
@@ -104,5 +104,5 @@
             <parent link="${name}_aligned_depth_to_fisheye1_frame"/>
             <child link="${name}_fisheye1_optical_frame"/>
-            <origin rpy="0 0 0" xyz="0.01 0 0"/>
+            <origin rpy="${M_PI/2} 0 -${M_PI/2}" xyz="0 0 0"/>
         </joint>
         <link name="${name}_fisheye1_optical_frame"/>
@@ -115,5 +115,5 @@
             <parent link="${name}_link"/>
             <child link="${name}_fisheye2_frame"/>
-            <origin rpy="0 0 0" xyz="0 -0.022 0"/>
+            <origin rpy="${M_PI} 0 ${M_PI}" xyz="0 -0.032 0"/>
         </joint>
         <link name="${name}_fisheye2_frame"/>
@@ -121,5 +121,5 @@
             <parent link="${name}_fisheye2_frame"/>
             <child link="${name}_fisheye2_optical_frame"/>
-            <origin rpy="0 0 0" xyz="0.01 0 0"/>
+            <origin rpy="${M_PI/2} 0 -${M_PI/2}" xyz="0 0 0"/>
         </joint>
         <link name="${name}_fisheye2_optical_frame"/>
@@ -132,5 +132,5 @@
             <parent link="${name}_link"/>
             <child link="${name}_gyro_frame"/>
-            <origin rpy="-${M_PI} 0 -${M_PI}" xyz="0 0.02 0"/>
+            <origin rpy="0 0 ${M_PI}" xyz="0 0.021 0"/>
         </joint>
         <link name="${name}_gyro_frame"/>
@@ -138,8 +138,32 @@
             <parent link="${name}_gyro_frame"/>
             <child link="${name}_gyro_optical_frame"/>
-            <origin rpy="-${M_PI/2} -${M_PI/2} 0" xyz="0 0 0"/>
+            <origin rpy="${M_PI/2} 0 -${M_PI/2}" xyz="0 0 0"/>
         </joint>
         <link name="${name}_gyro_optical_frame"/>
-        <gazebo reference="${name}_gyro_frame">
+        <joint name="${name}_accel_joint" type="fixed">
+            <parent link="${name}_link"/>
+            <child link="${name}_accel_frame"/>
+            <origin rpy="0 0 ${M_PI}" xyz="0 0.021 0"/>
+        </joint>
+        <link name="${name}_accel_frame"/>
+        <joint name="${name}_accel_optical_joint" type="fixed">
+            <parent link="${name}_accel_frame"/>
+            <child link="${name}_accel_optical_frame"/>
+            <origin rpy="${M_PI/2} 0 -${M_PI/2}" xyz="0 0 0"/>
+        </joint>
+        <link name="${name}_accel_optical_frame"/>
+        <joint name="${name}_imu_joint" type="fixed">
+            <parent link="${name}_link"/>
+            <child link="${name}_imu_frame"/>
+            <origin rpy="0 0 ${M_PI}" xyz="0 0.021 0"/>
+        </joint>
+        <link name="${name}_imu_frame"/>
+        <joint name="${name}_imu_optical_joint" type="fixed">
+            <parent link="${name}_imu_frame"/>
+            <child link="${name}_imu_optical_frame"/>
+            <origin rpy="${M_PI/2} 0 -${M_PI/2}" xyz="0 0 0"/>
+        </joint>
+        <link name="${name}_imu_optical_frame"/>
+        <gazebo reference="${name}_imu_optical_frame">
             <gravity>true</gravity>
             <sensor name="${name}_imu" type="imu">
@@ -151,5 +175,5 @@
                         <remapping>~/out:=camera/imu</remapping>
                     </ros>
-                    <frame_name>${name}_link</frame_name>
+                    <frame_name>${name}_imu_optical_frame</frame_name>
                 </plugin>
                 <imu>
@@ -209,16 +233,4 @@
             </sensor>
         </gazebo>
-        <joint name="${name}_accel_joint" type="fixed">
-            <parent link="${name}_link"/>
-            <child link="${name}_accel_frame"/>
-            <origin rpy="0 0 0" xyz="0 0.02 0"/>
-        </joint>
-        <link name="${name}_accel_frame"/>
-        <joint name="${name}_accel_optical_joint" type="fixed">
-            <parent link="${name}_accel_frame"/>
-            <child link="${name}_accel_optical_frame"/>
-            <origin rpy="-${M_PI/2} -${M_PI/2} 0" xyz="0 0 0"/>
-        </joint>
-        <link name="${name}_accel_optical_frame"/>
         <!-- odom -->
         <gazebo>
