Commit message: minor fix

File: vault_description/robots/vault.urdf.xacro (robot description, xacro)
@@ -5,6 +5,4 @@
     <xacro:include filename="$(find vault_description)/urdf/materials.xacro"/>
     <xacro:include filename="$(find vault_description)/urdf/box/vault_box.urdf.xacro" />
-    <xacro:include filename="$(find vault_description)/urdf/box/cover.urdf.xacro" />
-    <xacro:include filename="$(find vault_description)/urdf/box/realsense_mount.urdf.xacro" />
     <xacro:include filename="$(find vault_description)/urdf/sensors/all_sensors.urdf.xacro" />
     <!-- The base link -->
@@ -23,5 +21,3 @@
     <!-- box -->
     <xacro:vault_box parent="vault_link" />
-    <xacro:cover parent="vault_link" />
-    <xacro:realsense_mount parent="vault_link" />
 </robot>

File: vault_description/urdf/box/vault_box.urdf.xacro (robot description, xacro)
@@ -5,4 +5,6 @@
     <xacro:property name="box_depth" value="0.180" />
     <xacro:property name="box_mass" value="0.25" />
+    <xacro:include filename="$(find vault_description)/urdf/box/cover.urdf.xacro" />
+    <xacro:include filename="$(find vault_description)/urdf/box/realsense_mount.urdf.xacro" />
     <xacro:macro name="vault_box" params="parent">
         <link name="vault_box_link">
@@ -29,8 +31,10 @@
         </gazebo>
         <joint name="vault_box_joint" type="fixed">
-            <origin rpy="0 0 0" xyz="0 0 0"/>
+            <origin rpy="0 0 0" xyz="0 0 -0.01"/>
             <parent link="${parent}" />
             <child link="vault_box_link" />
         </joint>
+        <xacro:cover parent="vault_box_link" />
+        <xacro:realsense_mount parent="vault_box_link" />
     </xacro:macro>
 </robot>

Commit message: box fixed

File: vault_description/robots/vault.urdf.xacro (robot description, xacro)
@@ -5,4 +5,6 @@
     <xacro:include filename="$(find vault_description)/urdf/materials.xacro"/>
     <xacro:include filename="$(find vault_description)/urdf/box/vault_box.urdf.xacro" />
+    <xacro:include filename="$(find vault_description)/urdf/box/cover.urdf.xacro" />
+    <xacro:include filename="$(find vault_description)/urdf/box/realsense_mount.urdf.xacro" />
     <xacro:include filename="$(find vault_description)/urdf/sensors/all_sensors.urdf.xacro" />
     <!-- The base link -->
@@ -21,3 +23,5 @@
     <!-- box -->
     <xacro:vault_box parent="vault_link" />
+    <xacro:cover parent="vault_box_link" />
+    <xacro:realsense_mount parent="vault_box_link" />
 </robot>

File: vault_description/urdf/box/cover.urdf.xacro (robot description, xacro)
@@ -1,14 +1,14 @@
 <?xml version="1.0"?>
 <robot name="cover" xmlns:xacro="http://www.ros.org/wiki/xacro">
-    <xacro:property name="box_heigh" value="0.0085" />
-    <xacro:property name="box_width" value="0.168" />
-    <xacro:property name="box_depth" value="0.173" />
-    <xacro:property name="box_mass" value="0.1" />
     <xacro:macro name="cover" params="parent">
+        <xacro:property name="box_heigh" value="0.0085" />
+        <xacro:property name="box_width" value="0.168" />
+        <xacro:property name="box_depth" value="0.168" />
+        <xacro:property name="box_mass" value="0.01" />
         <link name="cover_link">
             <visual>
-                <origin rpy="0 0 0" xyz="0 0 0" />
+                <origin rpy="0 0 0" xyz="0 0.012 -0.015" />
                 <geometry>
-                    <mesh filename="package://vault_description/meshes/box/cover.stl"  scale="0.001 0.001 0.001"/>
+                    <mesh filename="package://vault_description/meshes/box/cover.stl" scale="0.001 0.001 0.001"/>
                 </geometry>
                 <material name="red" />
@@ -29,5 +29,5 @@
         </gazebo>
         <joint name="cover_joint" type="fixed">
-            <origin rpy="0 0 0" xyz="0 0 0"/>
+            <origin rpy="0 0 0" xyz="0 -0.012 -0.045"/>
             <parent link="${parent}" />
             <child link="cover_link" />

File: vault_description/urdf/box/realsense_mount.urdf.xacro (robot description, xacro)
@@ -1,12 +1,12 @@
 <?xml version="1.0"?>
 <robot name="realsense_mount" xmlns:xacro="http://www.ros.org/wiki/xacro">
-    <xacro:property name="box_heigh" value="0.033" />
-    <xacro:property name="box_width" value="0.080" />
-    <xacro:property name="box_depth" value="0.019" />
-    <xacro:property name="box_mass" value="0.1" />
     <xacro:macro name="realsense_mount" params="parent">
+        <xacro:property name="box_heigh" value="0.033" />
+        <xacro:property name="box_width" value="0.080" />
+        <xacro:property name="box_depth" value="0.019" />
+        <xacro:property name="box_mass" value="0.1" />
         <link name="realsense_mount_link">
             <visual>
-                <origin rpy="0 0 0" xyz="0 0 0" />
+                <origin rpy="0 0 0" xyz="0 0 -0.06" />
                 <geometry>
                     <mesh filename="package://vault_description/meshes/box/realsense_mount.stl"  scale="0.001 0.001 0.001"/>
@@ -14,10 +14,10 @@
                 <material name="green" />
             </visual>
-            <collision>
+            <!-- <collision>
                 <origin rpy="0 0 0" xyz="0 0 0" />
                 <geometry>
                     <box size="${box_width} ${box_depth} ${box_heigh}"/>
                 </geometry>
-            </collision>
+            </collision> -->
             <xacro:solid_cuboid_inertial
                 rpy="0 0 0" xyz="0 0 0"

File: vault_description/urdf/box/vault_box.urdf.xacro (robot description, xacro)
@@ -1,14 +1,12 @@
 <?xml version="1.0"?>
 <robot name="vault_box" xmlns:xacro="http://www.ros.org/wiki/xacro">
-    <xacro:property name="box_heigh" value="0.120" />
-    <xacro:property name="box_width" value="0.190" />
-    <xacro:property name="box_depth" value="0.180" />
-    <xacro:property name="box_mass" value="0.25" />
-    <xacro:include filename="$(find vault_description)/urdf/box/cover.urdf.xacro" />
-    <xacro:include filename="$(find vault_description)/urdf/box/realsense_mount.urdf.xacro" />
     <xacro:macro name="vault_box" params="parent">
+        <xacro:property name="box_heigh" value="0.120" />
+        <xacro:property name="box_width" value="0.190" />
+        <xacro:property name="box_depth" value="0.180" />
+        <xacro:property name="box_mass" value="0.25" />
         <link name="vault_box_link">
             <visual>
-                <origin rpy="0 0 0" xyz="0 0 0" />
+                <origin rpy="0 0 0" xyz="0 0 -0.06" />
                 <geometry>
                     <mesh filename="package://vault_description/meshes/box/vault_box.stl" scale="0.001 0.001 0.001"/>
@@ -31,10 +29,8 @@
         </gazebo>
         <joint name="vault_box_joint" type="fixed">
-            <origin rpy="0 0 0" xyz="0 0 -0.01"/>
+            <origin rpy="0 0 0" xyz="0 0 0"/>
             <parent link="${parent}" />
             <child link="vault_box_link" />
         </joint>
-        <xacro:cover parent="vault_box_link" />
-        <xacro:realsense_mount parent="vault_box_link" />
     </xacro:macro>
 </robot>

Commit message: realsense model added

File: vault_description/robots/vault.urdf.xacro (robot description, xacro)
@@ -24,4 +24,8 @@
     <xacro:vault_box parent="vault_link" />
     <xacro:cover parent="vault_box_link" />
-    <xacro:realsense_mount parent="vault_box_link" />
+    <xacro:realsense_mount parent="vault_link" />
+    <xacro:arg name="use_nominal_extrinsics" default="false" />
+    <xacro:sensor_d435i parent="realsense_mount_link" use_nominal_extrinsics="$(arg use_nominal_extrinsics)">
+        <origin xyz="0 -0.01 -0.005" rpy="0 0 -1.57"/>
+    </xacro:sensor_d435i>
 </robot>

File: vault_description/urdf/box/realsense_mount.urdf.xacro (robot description, xacro)
@@ -8,5 +8,5 @@
         <link name="realsense_mount_link">
             <visual>
-                <origin rpy="0 0 0" xyz="0 0 -0.06" />
+                <origin rpy="0 0 0" xyz="0.002 0.0775 -0.0526" />
                 <geometry>
                     <mesh filename="package://vault_description/meshes/box/realsense_mount.stl"  scale="0.001 0.001 0.001"/>
@@ -14,10 +14,10 @@
                 <material name="green" />
             </visual>
-            <!-- <collision>
+            <collision>
                 <origin rpy="0 0 0" xyz="0 0 0" />
                 <geometry>
                     <box size="${box_width} ${box_depth} ${box_heigh}"/>
                 </geometry>
-            </collision> -->
+            </collision>
             <xacro:solid_cuboid_inertial
                 rpy="0 0 0" xyz="0 0 0"
@@ -29,5 +29,5 @@
         </gazebo>
         <joint name="realsense_mount_joint" type="fixed">
-            <origin rpy="0 0 0" xyz="0 0 0"/>
+            <origin rpy="0 0 0" xyz="0 -0.0775 -0.0074"/>
             <parent link="${parent}" />
             <child link="realsense_mount_link" />

File: vault_description/urdf/materials.xacro (robot description, xacro)
@@ -1,5 +1,5 @@
 <?xml version="1.0" ?>
 <robot name="materials" xmlns:xacro="http://www.ros.org/wiki/xacro">
-   <material name="red">
+    <material name="red">
         <color rgba="0.8 0 0 1"/>
     </material>

File: vault_description/urdf/sensors/all_sensors.urdf.xacro (robot description, xacro)
@@ -7,3 +7,6 @@
   <!-- Hokuyo -->
   <xacro:include filename="$(find vault_description)/urdf/sensors/asus_xtion.urdf.xacro" />
+  <!-- Realsense -->
+  <xacro:include filename="$(find vault_description)/urdf/sensors/realsense/d435.urdf.xacro" />
+  <xacro:include filename="$(find vault_description)/urdf/sensors/realsense/d435i.urdf.xacro" />
 </robot>

Commit message: realsense mount fixed

File: vault_description/robots/vault.urdf.xacro (robot description, xacro)
@@ -27,5 +27,5 @@
     <xacro:arg name="use_nominal_extrinsics" default="false" />
     <xacro:sensor_d435i parent="realsense_mount_link" use_nominal_extrinsics="$(arg use_nominal_extrinsics)">
-        <origin xyz="0 -0.01 -0.005" rpy="0 0 -1.57"/>
+        <origin xyz="0 0 -0.005" rpy="0 0 -1.57"/>
     </xacro:sensor_d435i>
 </robot>

Commit message: vault simulated components added computer battery sensors (gps ublox, imu)

File: vault_description/robots/vault.urdf.xacro (robot description, xacro)
@@ -7,4 +7,6 @@
     <xacro:include filename="$(find vault_description)/urdf/box/cover.urdf.xacro" />
     <xacro:include filename="$(find vault_description)/urdf/box/realsense_mount.urdf.xacro" />
+    <xacro:include filename="$(find vault_description)/urdf/box/computer.urdf.xacro" />
+    <xacro:include filename="$(find vault_description)/urdf/box/battery.urdf.xacro" />
     <xacro:include filename="$(find vault_description)/urdf/sensors/all_sensors.urdf.xacro" />
     <!-- The base link -->
@@ -24,8 +26,20 @@
     <xacro:vault_box parent="vault_link" />
     <xacro:cover parent="vault_box_link" />
-    <xacro:realsense_mount parent="vault_link" />
+    <xacro:realsense_mount parent="vault_box_link" />
+    <xacro:computer parent="vault_box_link" />
+    <xacro:battery parent="vault_box_link" />
+    <!-- sensors -->
     <xacro:arg name="use_nominal_extrinsics" default="false" />
     <xacro:sensor_d435i parent="realsense_mount_link" use_nominal_extrinsics="$(arg use_nominal_extrinsics)">
         <origin xyz="0 0 -0.005" rpy="0 0 -1.57"/>
     </xacro:sensor_d435i>
+    <xacro:sensor_imu prefix="imu" parent="vault_box_link">
+        <origin xyz="0.075 -0.05 0" rpy="0 -1.57 0"/>
+    </xacro:sensor_imu>
+    <xacro:sensor_gps prefix="gps" parent="vault_box_link">
+        <origin xyz="0 0 0.0725" rpy="0 0 0"/>
+    </xacro:sensor_gps>
+    <xacro:gps_board prefix="gps" parent="vault_box_link">
+        <origin xyz="-0.072 -0.005 0" rpy="0 1.57 0"/>
+    </xacro:gps_board>
 </robot>

File: vault_description/urdf/box/vault_box.urdf.xacro (robot description, xacro)
@@ -4,5 +4,5 @@
         <xacro:property name="box_heigh" value="0.120" />
         <xacro:property name="box_width" value="0.190" />
-        <xacro:property name="box_depth" value="0.180" />
+        <xacro:property name="box_depth" value="0.210" />
         <xacro:property name="box_mass" value="0.25" />
         <link name="vault_box_link">

File: vault_description/urdf/materials.xacro (robot description, xacro)
@@ -9,4 +9,7 @@
     <material name="blue">
         <color rgba="0 0 0.8 1"/>
+    </material>
+    <material name="turquoise">
+        <color rgba="0.188 0.835 0.784 1"/>
     </material>
     <material name="orange">

File: vault_description/urdf/sensors/all_sensors.urdf.xacro (robot description, xacro)
@@ -5,6 +5,7 @@
   <!-- Hokuyo -->
   <xacro:include filename="$(find vault_description)/urdf/sensors/hokuyo.urdf.xacro" />
-  <!-- Hokuyo -->
-  <xacro:include filename="$(find vault_description)/urdf/sensors/asus_xtion.urdf.xacro" />
+  <!-- GPS -->
+  <xacro:include filename="$(find vault_description)/urdf/sensors/gps/gps.urdf.xacro" />
+  <xacro:include filename="$(find vault_description)/urdf/sensors/gps/gps_board.urdf.xacro" />
   <!-- Realsense -->
   <xacro:include filename="$(find vault_description)/urdf/sensors/realsense/d435.urdf.xacro" />

File: vault_description/urdf/sensors/imu.urdf.xacro (robot description, xacro)
@@ -17,17 +17,17 @@
         <origin rpy="0 0 0" xyz="0 0 0"/>
         <geometry>
-          <box size="0.03 0.02 0.01"/>
+          <box size="0.034 0.034 0.016"/>
         </geometry>
-        <material name="blue" />
+        <material name="turquoise" />
       </visual>
       <collision>
         <origin rpy="0 0 0" xyz="0 0 0"/>
         <geometry>
-          <box size=".001 .001 .001"/>
+          <box size="0.034 0.034 0.016"/>
         </geometry>
       </collision>
     </link>
     <gazebo reference="${prefix}_link">
-        <material>Gazebo/Blue</material>
+        <material>Gazebo/Turquoise</material>
     </gazebo>
     <gazebo reference="${prefix}_link">

File: vault_description/urdf/sensors/realsense/d435.urdf.xacro (robot description, xacro)
@@ -77,4 +77,7 @@
       </inertial>
     </link>
+    <gazebo reference="${name}_link">
+      <material>Gazebo/Silver</material>
+    </gazebo>
     <!-- Use the nominal extrinsics between camera frames if the calibrated extrinsics aren't being published. e.g. running the device in simulation  -->
     <xacro:if value="${use_nominal_extrinsics}">

Commit message: prefix and namspace added

File: vault_description/robots/vault.urdf.xacro (robot description, xacro)
@@ -11,5 +11,5 @@
     <xacro:include filename="$(find vault_description)/urdf/sensors/all_sensors.urdf.xacro" />
     <!-- The base link -->
-    <link name="vault_link">
+    <link name="base_link">
         <visual>
             <origin rpy="0 0 0" xyz="0 0 0" />
@@ -20,9 +20,9 @@
         </visual>
     </link>
-    <gazebo reference="vault_link">
+    <gazebo reference="base_link">
         <material>Gazebo/Orange</material>
     </gazebo>
     <!-- box -->
-    <xacro:vault_box parent="vault_link" />
+    <xacro:vault_box parent="base_link" />
     <xacro:cover parent="vault_box_link" />
     <xacro:realsense_mount parent="vault_box_link" />

File: vault_description/urdf/sensors/gps/gps.urdf.xacro (robot description, xacro)
@@ -2,4 +2,5 @@
 <robot name="sensor_gps" xmlns:xacro="http://www.ros.org/wiki/xacro">
   <xacro:macro name="sensor_gps" params="prefix parent *origin">
+    <xacro:arg name="prefix" default=""/>
     <!-- antenna -->
     <joint name="${prefix}_antenna_joint" type="fixed">
@@ -33,5 +34,5 @@
     </gazebo>
     <!-- plugin -->
-    <gazebo reference="gps_link">
+    <gazebo reference="${prefix}_antenna_link">
         <sensor name="gps_sensor" type="gps">
             <always_on>true</always_on>
@@ -41,8 +42,8 @@
                     <remapping>gps_controller/out:=gps</remapping>
                 </ros>
-                <frame_name>${prefix}_antenna_link</frame_name>
+                <frame_name>$(arg prefix)/${prefix}_antenna_link</frame_name>
             </plugin>
         </sensor>
-        <material>Gazebo/Silver</material>
+        <material>Gazebo/Grey</material>
     </gazebo>
   </xacro:macro>

File: vault_description/urdf/sensors/hokuyo.urdf.xacro (robot description, xacro)
@@ -2,4 +2,5 @@
 <robot name="sensor_hokuyo" xmlns:xacro="http://www.ros.org/wiki/xacro">
   <xacro:macro name="sensor_hokuyo" params="prefix parent *origin min_angle:=-1.57079637051 max_angle:=1.57079637051">
+    <xacro:arg name="prefix" default=""/>
     <joint name="${prefix}_base_joint" type="fixed">
       <xacro:insert_block name="origin" />
@@ -66,5 +67,5 @@
                   </ros>
                   <output_type>sensor_msgs/LaserScan</output_type>
-                  <frame_name>${prefix}_link</frame_name>
+                  <frame_name>$(arg prefix)/${prefix}_link</frame_name>
                 </plugin>
             </sensor>

File: vault_description/urdf/sensors/imu.urdf.xacro (robot description, xacro)
@@ -2,4 +2,5 @@
 <robot name="sensor_imu" xmlns:xacro="http://www.ros.org/wiki/xacro">
   <xacro:macro name="sensor_imu" params="prefix parent *origin">
+    <xacro:arg name="prefix" default=""/>
     <joint name="${prefix}_joint" type="fixed">
         <axis xyz="1 0 0"/>
@@ -38,5 +39,5 @@
           </ros>
           <initial_orientation_as_reference>false</initial_orientation_as_reference>
-          <frame_name>${prefix}_link</frame_name>
+          <frame_name>$(arg prefix)/${prefix}_link</frame_name>
         </plugin>
         <always_on>true</always_on>

File: vault_description/urdf/sensors/realsense/d435.urdf.xacro (robot description, xacro)
@@ -7,4 +7,5 @@
 -->
 <robot name="sensor_d435" xmlns:xacro="http://ros.org/wiki/xacro">
+  <xacro:arg name="prefix" default=""/>
   <xacro:macro name="sensor_d435" params="parent *origin name:=camera use_nominal_extrinsics:=false add_plug:=false use_mesh:=true">
     <!-- Includes -->
@@ -143,5 +144,5 @@
     <gazebo reference="${name}_link">
       <sensor name="${name}" type="depth">
-        <camera name="camera">
+        <camera name="${name}">
           <horizontal_fov>1.57</horizontal_fov>
           <image>
@@ -165,13 +166,13 @@
         <plugin name="camera_plugin" filename="libgazebo_ros_camera.so">
           <ros>
-            <remapping>/${name}/image_raw:=/${name}/color/image_raw</remapping>
-            <remapping>/${name}/image_raw/compressed:=/${name}/color/image_raw/compressed</remapping>
-            <remapping>/${name}/image_raw/compressedDepth:=/${name}/color/image_raw/compressedDepth</remapping>
-            <remapping>/${name}/camera_info:=/${name}/color/camera_info</remapping>
-            <remapping>/${name}/depth/image_raw:=/${name}/aligned_depth_to_color/image_raw</remapping>
-            <remapping>/${name}/depth/image_raw/compressed:=/${name}/aligned_depth_to_color/image_raw/compressed</remapping>
-            <remapping>/${name}/depth/image_raw/compressedDepth:=/${name}/aligned_depth_to_color/image_raw/compressedDepth</remapping>
-            <remapping>/${name}/depth/camera_info:=/${name}/aligned_depth_to_color/camera_info</remapping>
-            <remapping>/${name}/points:=/${name}/depth/color/points</remapping>
+            <remapping>/$(arg prefix)/${name}/image_raw:=/$(arg prefix)/${name}/color/image_raw</remapping>
+            <remapping>/$(arg prefix)/${name}/image_raw/compressed:=/$(arg prefix)/${name}/color/image_raw/compressed</remapping>
+            <remapping>/$(arg prefix)/${name}/image_raw/compressedDepth:=/$(arg prefix)/${name}/color/image_raw/compressedDepth</remapping>
+            <remapping>/$(arg prefix)/${name}/camera_info:=/$(arg prefix)/${name}/color/camera_info</remapping>
+            <remapping>/$(arg prefix)/${name}/depth/image_raw:=/$(arg prefix)/${name}/aligned_depth_to_color/image_raw</remapping>
+            <remapping>/$(arg prefix)/${name}/depth/image_raw/compressed:=/$(arg prefix)/${name}/aligned_depth_to_color/image_raw/compressed</remapping>
+            <remapping>/$(arg prefix)/${name}/depth/image_raw/compressedDepth:=/$(arg prefix)/${name}/aligned_depth_to_color/image_raw/compressedDepth</remapping>
+            <remapping>/$(arg prefix)/${name}/depth/camera_info:=/$(arg prefix)/${name}/aligned_depth_to_color/camera_info</remapping>
+            <remapping>/$(arg prefix)/${name}/points:=/$(arg prefix)/${name}/depth/color/points</remapping>
           </ros>
           <visualize>true</visualize>
@@ -179,5 +180,5 @@
           <always_on>true</always_on>
           <update_rate>0.0</update_rate>
-          <frame_name>${name}_color_optical_frame</frame_name>
+          <frame_name>$(arg prefix)/${name}_color_optical_frame</frame_name>
           <camera_name>camera</camera_name>
           <min_depth>0.3</min_depth>
