Commit message: minor fix to sensors

File: vault_description/robots/vault.urdf.xacro (robot description, xacro)
@@ -34,11 +34,11 @@
         <origin xyz="0 0 -0.005" rpy="0 0 -1.57"/>
     </xacro:sensor_d435i>
-    <xacro:sensor_imu prefix="imu" parent="vault_box_link">
+    <xacro:sensor_imu name="imu" parent="vault_box_link">
         <origin xyz="0.075 -0.05 0" rpy="0 -1.57 0"/>
     </xacro:sensor_imu>
-    <xacro:sensor_gps prefix="gps" parent="vault_box_link">
+    <xacro:sensor_gps name="gps" parent="vault_box_link">
         <origin xyz="0 0 0.0725" rpy="0 0 0"/>
     </xacro:sensor_gps>
-    <xacro:gps_board prefix="gps" parent="vault_box_link">
+    <xacro:gps_board name="gps" parent="vault_box_link">
         <origin xyz="-0.072 -0.005 0" rpy="0 1.57 0"/>
     </xacro:gps_board>

File: vault_description/urdf/sensors/all_sensors.urdf.xacro (robot description, xacro)
@@ -2,7 +2,7 @@
 <robot name="all_sensors" xmlns:xacro="http://www.ros.org/wiki/xacro">
   <!-- Imu -->
-  <xacro:include filename="$(find vault_description)/urdf/sensors/imu.urdf.xacro" />
+  <xacro:include filename="$(find vault_description)/urdf/sensors/imu/imu.urdf.xacro" />
   <!-- Hokuyo -->
-  <xacro:include filename="$(find vault_description)/urdf/sensors/hokuyo.urdf.xacro" />
+  <xacro:include filename="$(find vault_description)/urdf/sensors/hokuyo/hokuyo.urdf.xacro" />
   <!-- GPS -->
   <xacro:include filename="$(find vault_description)/urdf/sensors/gps/gps.urdf.xacro" />

File: vault_description/urdf/sensors/gps/gps.urdf.xacro (robot description, xacro)
@@ -1,14 +1,14 @@
 <?xml version="1.0"?>
 <robot name="sensor_gps" xmlns:xacro="http://www.ros.org/wiki/xacro">
-  <xacro:macro name="sensor_gps" params="prefix parent *origin">
+  <xacro:macro name="sensor_gps" params="name parent *origin">
     <xacro:arg name="prefix" default=""/>
     <!-- antenna -->
-    <joint name="${prefix}_antenna_joint" type="fixed">
+    <joint name="${name}_antenna_joint" type="fixed">
         <axis xyz="1 0 0"/>
         <xacro:insert_block name="origin"/>
         <parent link="${parent}"/>
-        <child link="${prefix}_antenna_link"/>
+        <child link="${name}_antenna_link"/>
     </joint>
-    <link name="${prefix}_antenna_link">
+    <link name="${name}_antenna_link">
       <inertial>
         <mass value="0.001"/>
@@ -30,9 +30,9 @@
       </collision>
     </link>
-    <gazebo reference="${prefix}_antenna_link">
+    <gazebo reference="${name}_antenna_link">
       <material>Gazebo/Grey</material>
     </gazebo>
     <!-- plugin -->
-    <gazebo reference="${prefix}_antenna_link">
+    <gazebo reference="${name}_antenna_link">
         <sensor name="gps_sensor" type="gps">
             <always_on>true</always_on>
@@ -40,7 +40,7 @@
             <plugin name="gps_controller" filename="libgazebo_ros_gps_sensor.so">
                 <ros>
-                    <remapping>gps_controller/out:=gps</remapping>
+                    <remapping>gps_controller/out:=fix</remapping>
                 </ros>
-                <frame_name>$(arg prefix)/${prefix}_antenna_link</frame_name>
+                <frame_name>$(arg prefix)/${name}_antenna_link</frame_name>
             </plugin>
         </sensor>

File: vault_description/urdf/sensors/gps/gps_board.urdf.xacro (robot description, xacro)
@@ -1,13 +1,13 @@
 <?xml version="1.0"?>
 <robot name="gps_board" xmlns:xacro="http://www.ros.org/wiki/xacro">
-  <xacro:macro name="gps_board" params="prefix parent *origin">
+  <xacro:macro name="gps_board" params="name parent *origin">
     <!-- board -->
-    <joint name="${prefix}_joint" type="fixed">
+    <joint name="${name}_joint" type="fixed">
         <axis xyz="1 0 0"/>
         <xacro:insert_block name="origin"/>
         <parent link="${parent}"/>
-        <child link="${prefix}_board_link"/>
+        <child link="${name}_board_link"/>
     </joint>
-    <link name="${prefix}_board_link">
+    <link name="${name}_board_link">
       <inertial>
         <mass value="0.001"/>
@@ -29,5 +29,5 @@
       </collision>
     </link>
-    <gazebo reference="${prefix}_board_link">
+    <gazebo reference="${name}_board_link">
       <material>Gazebo/Grey</material>
     </gazebo>

File: vault_description/urdf/sensors/hokuyo/hokuyo.urdf.xacro (robot description, xacro)
@@ -3,10 +3,10 @@
   <xacro:macro name="sensor_hokuyo" params="prefix parent *origin min_angle:=-1.57079637051 max_angle:=1.57079637051">
     <xacro:arg name="prefix" default=""/>
-    <joint name="${prefix}_base_joint" type="fixed">
+    <joint name="${name}_base_joint" type="fixed">
       <xacro:insert_block name="origin" />
       <parent link="${parent}"/>
-      <child link="${prefix}_base_link"/>
+      <child link="${name}_base_link"/>
     </joint>
-    <link name="${prefix}_base_link">
+    <link name="${name}_base_link">
       <collision>
         <origin xyz="0 0 -0.05" rpy="0 0 0"/>
@@ -27,15 +27,15 @@
       </inertial>
     </link>
-    <gazebo reference="${prefix}_base_link">
+    <gazebo reference="${name}_base_link">
         <material>Gazebo/DarkGrey</material>
     </gazebo>
-    <link name="${prefix}_link">
+    <link name="${name}_link">
     </link>
-    <joint name="${prefix}_joint" type="fixed">
-      <parent link="${prefix}_base_link"/>
-      <child link="${prefix}_link"/>
+    <joint name="${name}_joint" type="fixed">
+      <parent link="${name}_base_link"/>
+      <child link="${name}_link"/>
       <origin xyz="0.00 0 0.0" rpy="0 0 0"/>
     </joint>
-    <gazebo reference="${prefix}_link">
+    <gazebo reference="${name}_link">
             <sensor type="gpu_ray" name="hokuyo_sensor">
                 <pose>0 0 0 0 0 0</pose>
@@ -62,10 +62,10 @@
                     </noise>
                 </ray>
-                <plugin name="${prefix}_controller" filename="libgazebo_ros_ray_sensor.so">
+                <plugin name="${name}_controller" filename="libgazebo_ros_ray_sensor.so">
                   <ros>
                     <argument>~/out:=scan</argument>
                   </ros>
                   <output_type>sensor_msgs/LaserScan</output_type>
-                  <frame_name>$(arg prefix)/${prefix}_link</frame_name>
+                  <frame_name>$(arg prefix)/${name}_link</frame_name>
                 </plugin>
             </sensor>

File: vault_description/urdf/sensors/imu/imu.urdf.xacro (robot description, xacro)
@@ -1,13 +1,13 @@
 <?xml version="1.0"?>
 <robot name="sensor_imu" xmlns:xacro="http://www.ros.org/wiki/xacro">
-  <xacro:macro name="sensor_imu" params="prefix parent *origin">
+  <xacro:macro name="sensor_imu" params="name parent *origin">
     <xacro:arg name="prefix" default=""/>
-    <joint name="${prefix}_joint" type="fixed">
+    <joint name="${name}_joint" type="fixed">
         <axis xyz="1 0 0"/>
         <xacro:insert_block name="origin"/>
         <parent link="${parent}"/>
-        <child link="${prefix}_link"/>
+        <child link="${name}_link"/>
     </joint>
-    <link name="${prefix}_link">
+    <link name="${name}_link">
       <inertial>
         <mass value="0.001"/>
@@ -29,8 +29,8 @@
       </collision>
     </link>
-    <gazebo reference="${prefix}_link">
+    <gazebo reference="${name}_link">
         <material>Gazebo/Turquoise</material>
     </gazebo>
-    <gazebo reference="${prefix}_link">
+    <gazebo reference="${name}_link">
       <sensor name="imu_sensor" type="imu">
         <plugin filename="libgazebo_ros_imu_sensor.so" name="imu_controller">
@@ -39,5 +39,5 @@
           </ros>
           <initial_orientation_as_reference>false</initial_orientation_as_reference>
-          <frame_name>$(arg prefix)/${prefix}_link</frame_name>
+          <frame_name>$(arg prefix)/${name}_link</frame_name>
         </plugin>
         <always_on>true</always_on>

File: vault_description/urdf/sensors/realsense/d435.urdf.xacro (robot description, xacro)
@@ -166,13 +166,13 @@
         <plugin name="camera_plugin" filename="libgazebo_ros_camera.so">
           <ros>
-            <remapping>/$(arg prefix)/${name}/image_raw:=/$(arg prefix)/${name}/color/image_raw</remapping>
-            <remapping>/$(arg prefix)/${name}/image_raw/compressed:=/$(arg prefix)/${name}/color/image_raw/compressed</remapping>
-            <remapping>/$(arg prefix)/${name}/image_raw/compressedDepth:=/$(arg prefix)/${name}/color/image_raw/compressedDepth</remapping>
-            <remapping>/$(arg prefix)/${name}/camera_info:=/$(arg prefix)/${name}/color/camera_info</remapping>
-            <remapping>/$(arg prefix)/${name}/depth/image_raw:=/$(arg prefix)/${name}/aligned_depth_to_color/image_raw</remapping>
-            <remapping>/$(arg prefix)/${name}/depth/image_raw/compressed:=/$(arg prefix)/${name}/aligned_depth_to_color/image_raw/compressed</remapping>
-            <remapping>/$(arg prefix)/${name}/depth/image_raw/compressedDepth:=/$(arg prefix)/${name}/aligned_depth_to_color/image_raw/compressedDepth</remapping>
-            <remapping>/$(arg prefix)/${name}/depth/camera_info:=/$(arg prefix)/${name}/aligned_depth_to_color/camera_info</remapping>
-            <remapping>/$(arg prefix)/${name}/points:=/$(arg prefix)/${name}/depth/color/points</remapping>
+            <remapping>camera/image_raw:=camera/color/image_raw</remapping>
+            <remapping>camera/image_raw/compressed:=camera/color/image_raw/compressed</remapping>
+            <remapping>camera/image_raw/compressedDepth:=camera/color/image_raw/compressedDepth</remapping>
+            <remapping>camera/camera_info:=camera/color/camera_info</remapping>
+            <remapping>camera/depth/image_raw:=camera/aligned_depth_to_color/image_raw</remapping>
+            <remapping>camera/depth/image_raw/compressed:=camera/aligned_depth_to_color/image_raw/compressed</remapping>
+            <remapping>camera/depth/image_raw/compressedDepth:=camera/aligned_depth_to_color/image_raw/compressedDepth</remapping>
+            <remapping>camera/depth/camera_info:=camera/aligned_depth_to_color/camera_info</remapping>
+            <remapping>camera/points:=camera/depth/color/points</remapping>
           </ros>
           <visualize>true</visualize>

Commit message: tf namespace fixed vault/ -> vault_

File: vault_description/robots/vault.urdf.xacro (robot description, xacro)
@@ -4,5 +4,5 @@
     <xacro:include filename="$(find vault_description)/urdf/inertials.xacro"/>
     <xacro:include filename="$(find vault_description)/urdf/materials.xacro"/>
-    <xacro:include filename="$(find vault_description)/urdf/box/vault_box.urdf.xacro" />
+    <xacro:include filename="$(find vault_description)/urdf/box/box.urdf.xacro" />
     <xacro:include filename="$(find vault_description)/urdf/box/cover.urdf.xacro" />
     <xacro:include filename="$(find vault_description)/urdf/box/realsense_mount.urdf.xacro" />
@@ -11,5 +11,5 @@
     <xacro:include filename="$(find vault_description)/urdf/sensors/all_sensors.urdf.xacro" />
     <!-- The base link -->
-    <link name="base_link">
+    <link name="vault_base_link">
         <visual>
             <origin rpy="0 0 0" xyz="0 0 0" />
@@ -20,25 +20,25 @@
         </visual>
     </link>
-    <gazebo reference="base_link">
+    <gazebo reference="vault_base_link">
         <material>Gazebo/Orange</material>
     </gazebo>
     <!-- box -->
-    <xacro:vault_box parent="base_link" />
-    <xacro:cover parent="vault_box_link" />
-    <xacro:realsense_mount parent="vault_box_link" />
-    <xacro:computer parent="vault_box_link" />
-    <xacro:battery parent="vault_box_link" />
+    <xacro:vault_box parent="vault_base_link" />
+    <xacro:vault_cover parent="vault_box_link" />
+    <xacro:vault_realsense_mount parent="vault_box_link" />
+    <xacro:vault_computer parent="vault_box_link" />
+    <xacro:vault_battery parent="vault_box_link" />
     <!-- sensors -->
     <xacro:arg name="use_nominal_extrinsics" default="true" />
-    <xacro:sensor_d435i parent="realsense_mount_link" use_nominal_extrinsics="$(arg use_nominal_extrinsics)">
+    <xacro:sensor_d435i parent="vault_realsense_mount_link" name="vault_camera" use_nominal_extrinsics="$(arg use_nominal_extrinsics)">
         <origin xyz="0 0 -0.005" rpy="0 0 -1.57"/>
     </xacro:sensor_d435i>
-    <xacro:sensor_imu name="imu" parent="vault_box_link">
+    <xacro:sensor_imu name="vault_imu" parent="vault_box_link">
         <origin xyz="0.075 -0.05 0" rpy="0 -1.57 0"/>
     </xacro:sensor_imu>
-    <xacro:sensor_gps name="gps" parent="vault_box_link">
+    <xacro:sensor_gps name="vault_gps" parent="vault_box_link">
         <origin xyz="0 0 0.0725" rpy="0 0 0"/>
     </xacro:sensor_gps>
-    <xacro:gps_board name="gps" parent="vault_box_link">
+    <xacro:gps_board name="vault_gps" parent="vault_box_link">
         <origin xyz="-0.072 -0.005 0" rpy="0 1.57 0"/>
     </xacro:gps_board>

File: vault_description/urdf/box/battery.urdf.xacro (robot description, xacro)
@@ -1,10 +1,10 @@
 <?xml version="1.0"?>
-<robot name="battery" xmlns:xacro="http://www.ros.org/wiki/xacro">
-    <xacro:macro name="battery" params="parent">
+<robot name="vault_battery" xmlns:xacro="http://www.ros.org/wiki/xacro">
+    <xacro:macro name="vault_battery" params="parent">
         <xacro:property name="box_heigh" value="0.076" />
         <xacro:property name="box_width" value="0.158" />
         <xacro:property name="box_depth" value="0.038" />
         <xacro:property name="box_mass" value="1.000" />
-        <link name="battery_link">
+        <link name="vault_battery_link">
             <visual>
                 <origin rpy="0 0 0" xyz="0 0 0" />
@@ -25,11 +25,11 @@
                 x="${box_width}" y="${box_depth}" z="${box_heigh}" />
         </link>
-        <gazebo reference="battery_link">
+        <gazebo reference="vault_battery_link">
             <material>Gazebo/Blue</material>
         </gazebo>
-        <joint name="battery_joint" type="fixed">
+        <joint name="vault_battery_joint" type="fixed">
             <origin rpy="0 0 0" xyz="0 0.08 -0.002"/>
             <parent link="${parent}" />
-            <child link="battery_link" />
+            <child link="vault_battery_link" />
         </joint>
     </xacro:macro>

File: vault_description/urdf/box/box.urdf.xacro (robot description, xacro)
@@ -10,5 +10,5 @@
                 <origin rpy="0 0 0" xyz="0 0 -0.06" />
                 <geometry>
-                    <mesh filename="package://vault_description/meshes/box/vault_box.stl" scale="0.001 0.001 0.001"/>
+                    <mesh filename="package://vault_description/meshes/box/box.stl" scale="0.001 0.001 0.001"/>
                 </geometry>
                 <material name="black" />

File: vault_description/urdf/box/computer.urdf.xacro (robot description, xacro)
@@ -1,10 +1,10 @@
 <?xml version="1.0"?>
-<robot name="computer" xmlns:xacro="http://www.ros.org/wiki/xacro">
-    <xacro:macro name="computer" params="parent">
+<robot name="vault_computer" xmlns:xacro="http://www.ros.org/wiki/xacro">
+    <xacro:macro name="vault_computer" params="parent">
         <xacro:property name="box_heigh" value="0.040" />
         <xacro:property name="box_width" value="0.110" />
         <xacro:property name="box_depth" value="0.110" />
         <xacro:property name="box_mass" value="0.500" />
-        <link name="computer_link">
+        <link name="vault_computer_link">
             <visual>
                 <origin rpy="0 0 0" xyz="0 0 0" />
@@ -25,11 +25,11 @@
                 x="${box_width}" y="${box_depth}" z="${box_heigh}" />
         </link>
-        <gazebo reference="computer_link">
+        <gazebo reference="vault_computer_link">
             <material>Gazebo/DarkGrey</material>
         </gazebo>
-        <joint name="computer_joint" type="fixed">
+        <joint name="vault_computer_joint" type="fixed">
             <origin rpy="0 0 0" xyz="0 0 0.03"/>
             <parent link="${parent}" />
-            <child link="computer_link" />
+            <child link="vault_computer_link" />
         </joint>
     </xacro:macro>

File: vault_description/urdf/box/cover.urdf.xacro (robot description, xacro)
@@ -1,10 +1,10 @@
 <?xml version="1.0"?>
-<robot name="cover" xmlns:xacro="http://www.ros.org/wiki/xacro">
-    <xacro:macro name="cover" params="parent">
+<robot name="vault_cover" xmlns:xacro="http://www.ros.org/wiki/xacro">
+    <xacro:macro name="vault_cover" params="parent">
         <xacro:property name="box_heigh" value="0.0085" />
         <xacro:property name="box_width" value="0.168" />
         <xacro:property name="box_depth" value="0.168" />
         <xacro:property name="box_mass" value="0.01" />
-        <link name="cover_link">
+        <link name="vault_cover_link">
             <visual>
                 <origin rpy="0 0 0" xyz="0 0.012 -0.015" />
@@ -25,11 +25,11 @@
                 x="${box_width}" y="${box_depth}" z="${box_heigh}" />
         </link>
-        <gazebo reference="cover_link">
+        <gazebo reference="vault_cover_link">
             <material>Gazebo/Red</material>
         </gazebo>
-        <joint name="cover_joint" type="fixed">
+        <joint name="vault_cover_joint" type="fixed">
             <origin rpy="0 0 0" xyz="0 -0.012 -0.045"/>
             <parent link="${parent}" />
-            <child link="cover_link" />
+            <child link="vault_cover_link" />
         </joint>
     </xacro:macro>

File: vault_description/urdf/box/realsense_mount.urdf.xacro (robot description, xacro)
@@ -1,10 +1,10 @@
 <?xml version="1.0"?>
-<robot name="realsense_mount" xmlns:xacro="http://www.ros.org/wiki/xacro">
-    <xacro:macro name="realsense_mount" params="parent">
+<robot name="vault_realsense_mount" xmlns:xacro="http://www.ros.org/wiki/xacro">
+    <xacro:macro name="vault_realsense_mount" params="parent">
         <xacro:property name="box_heigh" value="0.033" />
         <xacro:property name="box_width" value="0.080" />
         <xacro:property name="box_depth" value="0.019" />
         <xacro:property name="box_mass" value="0.1" />
-        <link name="realsense_mount_link">
+        <link name="vault_realsense_mount_link">
             <visual>
                 <origin rpy="0 0 0" xyz="0.002 0.0775 -0.0526" />
@@ -25,11 +25,11 @@
                 x="${box_width}" y="${box_depth}" z="${box_heigh}" />
         </link>
-        <gazebo reference="realsense_mount_link">
+        <gazebo reference="vault_realsense_mount_link">
             <material>Gazebo/Green</material>
         </gazebo>
-        <joint name="realsense_mount_joint" type="fixed">
+        <joint name="vault_realsense_mount_joint" type="fixed">
             <origin rpy="0 0 0" xyz="0 -0.0775 -0.0074"/>
             <parent link="${parent}" />
-            <child link="realsense_mount_link" />
+            <child link="vault_realsense_mount_link" />
         </joint>
     </xacro:macro>

File: vault_description/urdf/sensors/gps/gps.urdf.xacro (robot description, xacro)
@@ -2,5 +2,4 @@
 <robot name="sensor_gps" xmlns:xacro="http://www.ros.org/wiki/xacro">
   <xacro:macro name="sensor_gps" params="name parent *origin">
-    <xacro:arg name="prefix" default=""/>
     <!-- antenna -->
     <joint name="${name}_antenna_joint" type="fixed">
@@ -42,5 +41,5 @@
                     <remapping>gps_controller/out:=fix</remapping>
                 </ros>
-                <frame_name>$(arg prefix)/${name}_antenna_link</frame_name>
+                <frame_name>${name}_antenna_link</frame_name>
             </plugin>
         </sensor>

File: vault_description/urdf/sensors/hokuyo/hokuyo.urdf.xacro (robot description, xacro)
@@ -2,5 +2,4 @@
 <robot name="sensor_hokuyo" xmlns:xacro="http://www.ros.org/wiki/xacro">
   <xacro:macro name="sensor_hokuyo" params="prefix parent *origin min_angle:=-1.57079637051 max_angle:=1.57079637051">
-    <xacro:arg name="prefix" default=""/>
     <joint name="${name}_base_joint" type="fixed">
       <xacro:insert_block name="origin" />
@@ -67,5 +66,5 @@
                   </ros>
                   <output_type>sensor_msgs/LaserScan</output_type>
-                  <frame_name>$(arg prefix)/${name}_link</frame_name>
+                  <frame_name>${name}_link</frame_name>
                 </plugin>
             </sensor>

File: vault_description/urdf/sensors/imu/imu.urdf.xacro (robot description, xacro)
@@ -2,5 +2,4 @@
 <robot name="sensor_imu" xmlns:xacro="http://www.ros.org/wiki/xacro">
   <xacro:macro name="sensor_imu" params="name parent *origin">
-    <xacro:arg name="prefix" default=""/>
     <joint name="${name}_joint" type="fixed">
         <axis xyz="1 0 0"/>
@@ -39,5 +38,5 @@
           </ros>
           <initial_orientation_as_reference>false</initial_orientation_as_reference>
-          <frame_name>$(arg prefix)/${name}_link</frame_name>
+          <frame_name>${name}_link</frame_name>
         </plugin>
         <always_on>true</always_on>

File: vault_description/urdf/sensors/realsense/d435.urdf.xacro (robot description, xacro)
@@ -7,5 +7,4 @@
 -->
 <robot name="sensor_d435" xmlns:xacro="http://ros.org/wiki/xacro">
-  <xacro:arg name="prefix" default=""/>
   <xacro:macro name="sensor_d435" params="parent *origin name:=camera use_nominal_extrinsics:=false add_plug:=false use_mesh:=true">
     <!-- Includes -->
@@ -180,5 +179,5 @@
           <always_on>true</always_on>
           <update_rate>0.0</update_rate>
-          <frame_name>$(arg prefix)/${name}_color_optical_frame</frame_name>
+          <frame_name>${name}_color_optical_frame</frame_name>
           <camera_name>camera</camera_name>
           <min_depth>0.3</min_depth>
