Commit message: new box models

File: vault_description/robots/vault.urdf.xacro (robot description, xacro)
@@ -32,5 +32,5 @@
     <xacro:arg name="use_nominal_extrinsics" default="true" />
     <xacro:sensor_d435i parent="vault_realsense_mount_link" name="vault_camera" use_nominal_extrinsics="$(arg use_nominal_extrinsics)">
-        <origin xyz="0 0 -0.005" rpy="0 0 -1.57"/>
+        <origin xyz="0 -0.005 -0.005" rpy="0 0 -1.57"/>
     </xacro:sensor_d435i>
     <xacro:sensor_imu name="vault_imu" parent="vault_box_link">
@@ -38,5 +38,5 @@
     </xacro:sensor_imu>
     <xacro:sensor_gps name="vault_gps" parent="vault_box_link">
-        <origin xyz="0 0 0.0725" rpy="0 0 0"/>
+        <origin xyz="0 0 0.1025" rpy="0 0 0"/>
     </xacro:sensor_gps>
     <xacro:gps_board name="vault_gps" parent="vault_box_link">

File: vault_description/urdf/box/computer.urdf.xacro (robot description, xacro)
@@ -29,5 +29,5 @@
         </gazebo>
         <joint name="vault_computer_joint" type="fixed">
-            <origin rpy="0 0 0" xyz="0 0 0.03"/>
+            <origin rpy="0 0 0" xyz="0 0 0.060"/>
             <parent link="${parent}" />
             <child link="vault_computer_link" />

File: vault_description/urdf/box/cover.urdf.xacro (robot description, xacro)
@@ -4,9 +4,9 @@
         <xacro:property name="box_heigh" value="0.0085" />
         <xacro:property name="box_width" value="0.168" />
-        <xacro:property name="box_depth" value="0.168" />
+        <xacro:property name="box_depth" value="0.213" />
         <xacro:property name="box_mass" value="0.01" />
         <link name="vault_cover_link">
             <visual>
-                <origin rpy="0 0 0" xyz="0 0.012 -0.015" />
+                <origin rpy="0 0 0" xyz="0 -0.008 -0.015" />
                 <geometry>
                     <mesh filename="package://vault_description/meshes/box/cover.stl" scale="0.001 0.001 0.001"/>
@@ -29,5 +29,5 @@
         </gazebo>
         <joint name="vault_cover_joint" type="fixed">
-            <origin rpy="0 0 0" xyz="0 -0.012 -0.045"/>
+            <origin rpy="0 0 0" xyz="0 0.006 -0.0445"/>
             <parent link="${parent}" />
             <child link="vault_cover_link" />

File: vault_description/urdf/box/realsense_mount.urdf.xacro (robot description, xacro)
@@ -4,9 +4,9 @@
         <xacro:property name="box_heigh" value="0.033" />
         <xacro:property name="box_width" value="0.080" />
-        <xacro:property name="box_depth" value="0.019" />
+        <xacro:property name="box_depth" value="0.030" />
         <xacro:property name="box_mass" value="0.1" />
         <link name="vault_realsense_mount_link">
             <visual>
-                <origin rpy="0 0 0" xyz="0.002 0.0775 -0.0526" />
+                <origin rpy="0 0 0" xyz="0.002 0.069 -0.0675" />
                 <geometry>
                     <mesh filename="package://vault_description/meshes/box/realsense_mount.stl"  scale="0.001 0.001 0.001"/>
@@ -29,5 +29,5 @@
         </gazebo>
         <joint name="vault_realsense_mount_joint" type="fixed">
-            <origin rpy="0 0 0" xyz="0 -0.0775 -0.0074"/>
+            <origin rpy="0 0 0" xyz="0 -0.0695 0.0075"/>
             <parent link="${parent}" />
             <child link="vault_realsense_mount_link" />

Commit message: frames fixed

File: vault_description/robots/vault.urdf.xacro (robot description, xacro)
@@ -1,45 +1,9 @@
 <?xml version="1.0" ?>
 <robot name="vault" xmlns:xacro="http://www.ros.org/wiki/xacro">
-    <!-- Include macros -->
-    <xacro:include filename="$(find vault_description)/urdf/inertials.xacro"/>
+    <xacro:include filename="$(find vault_description)/urdf/vault.urdf.xacro"/>
     <xacro:include filename="$(find vault_description)/urdf/materials.xacro"/>
-    <xacro:include filename="$(find vault_description)/urdf/box/box.urdf.xacro" />
-    <xacro:include filename="$(find vault_description)/urdf/box/cover.urdf.xacro" />
-    <xacro:include filename="$(find vault_description)/urdf/box/realsense_mount.urdf.xacro" />
-    <xacro:include filename="$(find vault_description)/urdf/box/computer.urdf.xacro" />
-    <xacro:include filename="$(find vault_description)/urdf/box/battery.urdf.xacro" />
-    <xacro:include filename="$(find vault_description)/urdf/sensors/all_sensors.urdf.xacro" />
-    <!-- The base link -->
-    <link name="vault_base_link">
-        <visual>
-            <origin rpy="0 0 0" xyz="0 0 0" />
-            <geometry>
-                <box size="0.01 0.01 0.01"/>
-            </geometry>
-            <material name="orange" />
-        </visual>
-    </link>
-    <gazebo reference="vault_base_link">
-        <material>Gazebo/Orange</material>
-    </gazebo>
-    <!-- box -->
-    <xacro:vault_box parent="vault_base_link" />
-    <xacro:vault_cover parent="vault_box_link" />
-    <xacro:vault_realsense_mount parent="vault_box_link" />
-    <xacro:vault_computer parent="vault_box_link" />
-    <xacro:vault_battery parent="vault_box_link" />
-    <!-- sensors -->
-    <xacro:arg name="use_nominal_extrinsics" default="true" />
-    <xacro:sensor_d435i parent="vault_realsense_mount_link" name="vault_camera" use_nominal_extrinsics="$(arg use_nominal_extrinsics)">
-        <origin xyz="0 -0.005 -0.005" rpy="0 0 -1.57"/>
-    </xacro:sensor_d435i>
-    <xacro:sensor_imu name="vault_imu" parent="vault_box_link">
-        <origin xyz="0.075 -0.05 0" rpy="0 -1.57 0"/>
-    </xacro:sensor_imu>
-    <xacro:sensor_gps name="vault_gps" parent="vault_box_link">
-        <origin xyz="0 0 0.1025" rpy="0 0 0"/>
-    </xacro:sensor_gps>
-    <xacro:gps_board name="vault_gps" parent="vault_box_link">
-        <origin xyz="-0.072 -0.005 0" rpy="0 1.57 0"/>
-    </xacro:gps_board>
+    <link name="base_link"/>
+    <xacro:vault parent="base_link">
+        <origin xyz="0 0 0" rpy="0 0 0"/>
+    </xacro:vault>
 </robot>

File: vault_description/urdf/sensors/realsense/d435.urdf.xacro (robot description, xacro)
@@ -144,5 +144,5 @@
       <sensor name="${name}" type="depth">
         <always_on>true</always_on>
-        <update_rate>30</update_rate>
+        <update_rate>60</update_rate>
         <visualize>false</visualize>
         <camera name="${name}">
