Commit message: initial urdf/gazebo

File: vault_description/urdf/sensors/all_sensors.urdf.xacro (robot description, xacro)
@@ -2,8 +2,8 @@
 <robot name="all_sensors" xmlns:xacro="http://www.ros.org/wiki/xacro">
   <!-- Imu -->
-  <xacro:include filename="$(find rover_description)/urdf/sensors/imu.urdf.xacro" />
+  <xacro:include filename="$(find vault_description)/urdf/sensors/imu.urdf.xacro" />
   <!-- Hokuyo -->
-  <xacro:include filename="$(find rover_description)/urdf/sensors/hokuyo.urdf.xacro" />
+  <xacro:include filename="$(find vault_description)/urdf/sensors/hokuyo.urdf.xacro" />
   <!-- Hokuyo -->
-  <xacro:include filename="$(find rover_description)/urdf/sensors/asus_xtion.urdf.xacro" />
+  <xacro:include filename="$(find vault_description)/urdf/sensors/asus_xtion.urdf.xacro" />
 </robot>

File: vault_description/urdf/sensors/asus_xtion.urdf.xacro (robot description, xacro)
@@ -13,5 +13,5 @@
         <origin rpy="${math_pi_over_2} 0 ${math_pi_over_2}" xyz="0 0 0"/>
         <geometry>
-          <mesh filename="package://rover_description/meshes/sensors/asus_xtion/asus_xtion_pro_live.dae" scale="0.001 0.001 0.001"/>
+          <mesh filename="package://vault_description/meshes/sensors/asus_xtion/asus_xtion_pro_live.dae" scale="0.001 0.001 0.001"/>
         </geometry>
       </visual>
@@ -19,5 +19,5 @@
         <origin rpy="${math_pi_over_2} 0 ${math_pi_over_2}" xyz="0 0 0"/>
         <geometry>
-          <mesh filename="package://rover_description/meshes/sensors/asus_xtion/asus_xtion_pro_live.dae" scale="0.001 0.001 0.001"/>
+          <mesh filename="package://vault_description/meshes/sensors/asus_xtion/asus_xtion_pro_live.dae" scale="0.001 0.001 0.001"/>
         </geometry>
       </collision>

File: vault_description/urdf/sensors/hokuyo.urdf.xacro (robot description, xacro)
@@ -17,5 +17,5 @@
         <origin xyz="0 0 -0.05" rpy="0 0 0"/>
         <geometry>
-            <mesh filename="package://rover_description/meshes/sensors/hokuyo/hokuyo_ust_20lx.dae"/>
+            <mesh filename="package://vault_description/meshes/sensors/hokuyo/hokuyo_ust_20lx.dae"/>
         </geometry>
       </visual>

Commit message: t265 started

File: vault_description/urdf/sensors/all_sensors.urdf.xacro (robot description, xacro)
@@ -11,3 +11,4 @@
   <xacro:include filename="$(find vault_description)/urdf/sensors/realsense/d435.urdf.xacro" />
   <xacro:include filename="$(find vault_description)/urdf/sensors/realsense/d435i.urdf.xacro" />
+  <xacro:include filename="$(find vault_description)/urdf/sensors/realsense/t265.urdf.xacro" />
 </robot>

File: vault_description/urdf/sensors/realsense/d435i_imu_modules.urdf.xacro (robot description, xacro)
@@ -46,4 +46,72 @@
         <child link="${name}_imu_optical_frame" />
       </joint>
+      <gazebo reference="${name}_imu_optical_frame">
+        <sensor name="camera_imu_sensor" type="imu">
+          <plugin filename="libgazebo_ros_imu_sensor.so" name="imu_controller">
+            <ros>
+              <remapping>~/out:=camera/imu</remapping>
+            </ros>
+            <initial_orientation_as_reference>false</initial_orientation_as_reference>
+            <frame_name>${name}_imu_optical_frame</frame_name>
+          </plugin>
+          <always_on>true</always_on>
+          <update_rate>200</update_rate>
+          <visualize>true</visualize>
+          <imu>
+            <angular_velocity>
+              <x>
+                <noise type="gaussian">
+                  <mean>0.0</mean>
+                  <stddev>2e-4</stddev>
+                  <bias_mean>0.0000075</bias_mean>
+                  <bias_stddev>0.0000008</bias_stddev>
+                </noise>
+              </x>
+              <y>
+                <noise type="gaussian">
+                  <mean>0.0</mean>
+                  <stddev>2e-4</stddev>
+                  <bias_mean>0.0000075</bias_mean>
+                  <bias_stddev>0.0000008</bias_stddev>
+                </noise>
+              </y>
+              <z>
+                <noise type="gaussian">
+                  <mean>0.0</mean>
+                  <stddev>2e-4</stddev>
+                  <bias_mean>0.0000075</bias_mean>
+                  <bias_stddev>0.0000008</bias_stddev>
+                </noise>
+              </z>
+            </angular_velocity>
+            <linear_acceleration>
+              <x>
+                <noise type="gaussian">
+                  <mean>0.0</mean>
+                  <stddev>1.7e-2</stddev>
+                  <bias_mean>0.1</bias_mean>
+                  <bias_stddev>0.001</bias_stddev>
+                </noise>
+              </x>
+              <y>
+                <noise type="gaussian">
+                  <mean>0.0</mean>
+                  <stddev>1.7e-2</stddev>
+                  <bias_mean>0.1</bias_mean>
+                  <bias_stddev>0.001</bias_stddev>
+                </noise>
+              </y>
+              <z>
+                <noise type="gaussian">
+                  <mean>0.0</mean>
+                  <stddev>1.7e-2</stddev>
+                  <bias_mean>0.1</bias_mean>
+                  <bias_stddev>0.001</bias_stddev>
+                </noise>
+              </z>
+            </linear_acceleration>
+          </imu>
+        </sensor>
+      </gazebo>
     </xacro:if>
   </xacro:macro>

File: vault_description/urdf/vault.urdf.xacro (robot description, xacro)
@@ -41,4 +41,7 @@
             <origin xyz="0 -0.005 -0.0075" rpy="0 0 -1.57"/>
         </xacro:sensor_d435i>
+        <!-- <xacro:sensor_t265 name="vault_camera" parent="vault_realsense_mount_link" rate="30">
+            <origin xyz="0 -0.01 0.0075" rpy="0 0 -1.57"/>
+        </xacro:sensor_t265> -->
         <xacro:sensor_imu name="vault_imu" parent="vault_box_link">
             <origin xyz="0 -0.075 0.084" rpy="0 -3.141516 0"/>
