Commit message: use_t265 added to vault description

File: vault_description/urdf/vault.urdf.xacro (robot description, xacro)
@@ -2,4 +2,5 @@
 <robot name="vault" xmlns:xacro="http://www.ros.org/wiki/xacro">
     <xacro:macro name="vault" params="parent *origin">
+        <xacro:arg name="t265" default="false"/>
         <!-- Include macros -->
         <xacro:include filename="$(find vault_description)/urdf/inertials.xacro"/>
@@ -37,11 +38,15 @@
         <xacro:vault_battery parent="vault_box_link" />
         <!-- sensors -->
-        <!-- <xacro:arg name="use_nominal_extrinsics" default="true" />
-        <xacro:sensor_d435i parent="vault_realsense_mount_link" name="vault_camera" use_nominal_extrinsics="$(arg use_nominal_extrinsics)">
-            <origin xyz="0 -0.005 -0.0075" rpy="0 0 -1.57"/>
-        </xacro:sensor_d435i> -->
-        <xacro:sensor_t265 name="vault_camera" parent="vault_realsense_mount_link" rate="30">
-            <origin xyz="0 -0.01 0.0075" rpy="0 0 -1.57"/>
-        </xacro:sensor_t265>
+        <xacro:unless value="$(arg t265)">
+            <xacro:arg name="use_nominal_extrinsics" default="true" />
+            <xacro:sensor_d435i parent="vault_realsense_mount_link" name="vault_camera" use_nominal_extrinsics="$(arg use_nominal_extrinsics)">
+                <origin xyz="0 -0.005 -0.0075" rpy="0 0 -1.57"/>
+            </xacro:sensor_d435i>
+        </xacro:unless>
+        <xacro:if value="$(arg t265)">
+            <xacro:sensor_t265 name="vault_camera" parent="vault_realsense_mount_link" rate="30">
+                <origin xyz="0 -0.01 0.0075" rpy="0 0 -1.57"/>
+            </xacro:sensor_t265>
+        </xacro:if>
         <xacro:sensor_imu name="vault_imu" parent="vault_box_link">
             <origin xyz="0 -0.075 0.084" rpy="0 -3.141516 0"/>

Commit message: imu pose fixed

File: vault_description/urdf/vault.urdf.xacro (robot description, xacro)
@@ -2,4 +2,5 @@
 <robot name="vault" xmlns:xacro="http://www.ros.org/wiki/xacro">
     <xacro:macro name="vault" params="parent *origin">
+        <xacro:property name="M_PI" value="3.1415926535897931" />
         <!-- Include macros -->
         <xacro:include filename="$(find vault_description)/urdf/inertials.xacro"/>
@@ -38,11 +39,11 @@
         <!-- sensors -->
         <xacro:sensor_d435i parent="vault_realsense_mount_link" name="d435i" namespace="vault">
-            <origin xyz="0 -0.005 -0.0075" rpy="0 0 -1.57"/>
+            <origin xyz="0 -0.005 -0.0075" rpy="0 0 -${M_PI/2}"/>
         </xacro:sensor_d435i>
         <xacro:sensor_t265 parent="vault_realsense_mount_link" name="t265" namespace="vault" base_link="${parent}">
-            <origin xyz="0 0.0035 0.035" rpy="0 0 -1.57"/>
+            <origin xyz="0 0.0035 0.035" rpy="0 0 -${M_PI/2}"/>
         </xacro:sensor_t265>
         <xacro:sensor_imu name="imu" namespace="vault" parent="vault_box_link">
-            <origin xyz="0 -0.075 0.084" rpy="0 -3.141516 0"/>
+            <origin xyz="0 -0.075 0.084" rpy="0 -${M_PI} ${M_PI/2}"/>
         </xacro:sensor_imu>
         <xacro:sensor_gps name="gps" namespace="vault" parent="vault_box_link">
@@ -50,5 +51,5 @@
         </xacro:sensor_gps>
         <xacro:gps_board name="gps" namespace="vault" parent="vault_box_link">
-            <origin xyz="-0.077 0 -0.010" rpy="1.57 0 1.57"/>
+            <origin xyz="-0.077 0 -0.010" rpy="${M_PI/2} 0 ${M_PI/2}"/>
         </xacro:gps_board>
     </xacro:macro>
